File: TBSEQ_Board_V1/HT16K33Panel/HT16K33Panel/HT16K33.kicad_sch (KiCad schematic)
At the start: 19 parts, among them IC1 HT16K33_28SOP-A_, J1 Conn_01x05_Pin

Commit message: HT16K33 Control
Parts:
- removed J1: Conn_01x05_Pin, Connector_PinHeader_2.54mm:PinHeader_1x05_P2.54mm_Vertical, symbol Connector:Conn_01x05_Pin
- renumbered IC1 to U7
