File: TBSEQ_Board_V1/HT16K33Panel/HT16K33Panel/HT16K33Panel.kicad_sch (KiCad schematic)
At the start: 0 parts

Commit message: HT16K33 Control
Other:
- added sheet CV (CV.kicad_sch)
- added sheet FRAM (FRAM.kicad_sch)
- added sheet Jack (Jack.kicad_sch)
- added sheet LevelConvert (LevelConvert.kicad_sch)
- added sheet MIDI_RX (MIDI_RX.kicad_sch)
- added sheet Power (Power.kicad_sch)
- added sheet RasPiPico (RasPiPico.kicad_sch)
- added sheet TEMPO (TEMPO.kicad_sch)
