File: TBSEQ_Board_V1/HT16K33Panel/HT16K33Panel/HT16K33Panel.kicad_pcb (KiCad board)
At the start: 2 copper layers, 200 x 90 mm, 85 parts, among them IC1 HT16K33_28SOP-A_, J1 Conn_01x05_Pin

Commit message: HT16K33 Control
Parts:
- added C2: 0.047uF, Capacitor_THT:C_Rect_L7.0mm_W2.5mm_P5.00mm, F.Cu at (167.9, 75.8)
- added C3: 0.1uF, Capacitor_THT:C_Rect_L7.0mm_W2.0mm_P5.00mm, F.Cu at (97.6, 53.0)
- added D36: 1SS120TD, Diode_THT:D_A-405_P2.54mm_Vertical_AnodeUp, F.Cu at (96.6, 40.0)
- added J10: Conn_01x04_Socket, Connector_PinHeader_2.54mm:PinHeader_1x04_P2.54mm_Vertical, F.Cu at (159.4, 39.8)
- added J11: Conn_01x04_Socket, Connector_PinHeader_2.54mm:PinHeader_1x04_P2.54mm_Vertical, F.Cu at (116.9, 32.2)
- added J12: Conn_01x08_Pin, Connector_PinHeader_2.54mm:PinHeader_1x08_P2.54mm_Vertical, F.Cu at (183.9, 48.2)
- added J13: Conn_01x02_Pin, Connector_PinHeader_2.54mm:PinHeader_1x02_P2.54mm_Vertical, F.Cu at (179.2, 61.2)
- added J14: Conn_01x04_Pin, Connector_PinSocket_2.54mm:PinSocket_1x04_P2.54mm_Vertical, F.Cu at (208.6, 48.3)
- added J15: Conn_01x03_Pin, Connector_PinHeader_2.54mm:PinHeader_1x03_P2.54mm_Vertical, F.Cu at (83.8, 52.8)
- added J2: Conn_01x02_Socket, Connector_PinHeader_2.54mm:PinHeader_1x02_P2.54mm_Vertical, F.Cu at (152.3, 24.2)
- added J3: Conn_01x04_Pin, Connector_PinSocket_2.54mm:PinSocket_1x04_P2.54mm_Vertical, F.Cu at (188.2, 48.2)
- added J4: Conn_01x02_Pin, Connector_PinHeader_2.54mm:PinHeader_1x02_P2.54mm_Vertical, F.Cu at (131.2, 30.4)
- added J5: Conn_01x02_Pin, Connector_PinHeader_2.54mm:PinHeader_1x02_P2.54mm_Vertical, F.Cu at (131.0, 37.9)
- added J6: Conn_01x04_Socket, Connector_PinHeader_2.54mm:PinHeader_1x04_P2.54mm_Vertical, F.Cu at (131.0, 50.7)
- added J7: Conn_01x04_Socket, Connector_PinHeader_2.54mm:PinHeader_1x04_P2.54mm_Vertical, F.Cu at (131.0, 63.4)
- added J8: Conn_01x02_Pin, Connector_PinHeader_2.54mm:PinHeader_1x02_P2.54mm_Vertical, F.Cu at (131.0, 76.2)
- added J9: Conn_01x02_Pin, Connector_PinHeader_2.54mm:PinHeader_1x02_P2.54mm_Vertical, F.Cu at (158.4, 64.8)
- added R14: 1K, Resistor_THT:R_Axial_DIN0207_L6.3mm_D2.5mm_P7.62mm_Horizontal, F.Cu at (121.4, 32.2)
- added R15: 1K, Resistor_THT:R_Axial_DIN0207_L6.3mm_D2.5mm_P7.62mm_Horizontal, F.Cu at (125.2, 32.2)
- added R16: 22K, Resistor_THT:R_Axial_DIN0207_L6.3mm_D2.5mm_P7.62mm_Horizontal, F.Cu at (164.7, 73.2)
- added R17: 10K, Resistor_THT:R_Axial_DIN0207_L6.3mm_D2.5mm_P7.62mm_Horizontal, F.Cu at (184.9, 80.8)
- added R18: 5.1K, Resistor_THT:R_Axial_DIN0207_L6.3mm_D2.5mm_P7.62mm_Horizontal, F.Cu at (181.7, 80.8)
- added R19: 220, Resistor_THT:R_Axial_DIN0207_L6.3mm_D2.5mm_P7.62mm_Horizontal, F.Cu at (83.0, 44.8)
- added R20: 220, Resistor_THT:R_Axial_DIN0207_L6.3mm_D2.5mm_P7.62mm_Horizontal, F.Cu at (82.8, 48.5)
- added S35: B3F-1000S, SamacSys_Parts:B3F1060, F.Cu at (169.6, 44.5)
- added U1: Raspberry Pi Pico DIP-40, SamacSys_Parts:Raspberry Pi Pico DIP-40_W17.76mm, F.Cu at (144.8, 30.0)
- added U2: IRLML6402(DIP6Convert), Package_DIP:DIP-6_W7.62mm, F.Cu at (158.9, 30.5)
- added U3: FM24CL16B(DIP8 Convert), Package_DIP:CERDIP-8_W7.62mm_SideBrazed_Socket, F.Cu at (114.6, 49.4)
- added U4: AE-LCNV4-MOSFET, SamacSys_Parts:CERDIP-14_W10.16mm_SideBrazed_LongPads_Socket, F.Cu at (198.7, 48.4)
- added U5: 74HC126, Package_DIP:DIP-14_W7.62mm, F.Cu at (165.1, 52.0)
- added U6: LM358, Package_DIP:DIP-8_W7.62mm, F.Cu at (171.1, 72.7)
- added U8: TLP2304_TPR,E, SamacSys_Parts:SOIC127P700X230-6N, F.Cu at (95.3, 46.5)
- added VR1: RK09D117000B, SamacSys_Parts:RK09D117000B, F.Cu at (197.3, 79.8)
- J1: value Conn_01x05_Pin -> KDJ03-5; footprint Connector_PinHeader_2.54mm:PinHeader_1x05_P2.54mm_Vertical -> SamacSys_Parts:KDJ035
- moved D24 47.9 mm to (74.4, 125.0)
- moved S22 47.5 mm to (76.1, 133.8)
- moved S23 47.4 mm to (76.1, 112.8)
- moved D4 45.9 mm to (85.4, 135.8)
- moved S1 45.8 mm to (87.3, 144.5)
- moved S2 45.0 mm to (93.6, 125.2)
- moved D5 44.8 mm to (91.6, 116.5)
- moved S3 42.2 mm to (98.1, 144.5)
- moved D6 42.1 mm to (96.2, 135.8)
- moved S4 41.4 mm to (104.3, 125.2)
- moved D7 41.4 mm to (102.4, 116.5)
- moved S7 41.2 mm to (132.8, 125.2)
- moved D10 41.0 mm to (130.9, 116.5)
- moved S5 38.6 mm to (108.8, 144.5)
- moved D8 38.4 mm to (106.9, 135.8)
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- renumbered IC1 to U7
Connections:
- J1 pad 1: D+5V -> unconnected-(J1-Pad1)
- J1 pad 2: D+3.3V -> unconnected-(J1-Pad2)
- J1 pad 3: D_I2C_SCL -> unconnected-(J1-Pad3)
- J1 pad 4: D_I2C_SDA -> Net-(J1-Pad4)
- J1 pad 5: GNDD -> Net-(D36-A)
Routing:
- net D+3.3V: track 16.3 -> 205.8 mm, vias 0 -> 1
- net D+5V: track 0.00 -> 105.0 mm
- net Row15: track 224.5 -> 158.2 mm, vias 0 -> 1
- net Row3: track 223.2 -> 159.1 mm, vias 1 -> 2
- net Row2: track 221.5 -> 158.5 mm, vias 1 -> 2
- net A+TEMPO: track 0.00 -> 62.8 mm
- net D_I2C_SCL: track 9.29 -> 61.0 mm
- net D_I2C_SDA: track 13.1 -> 64.1 mm, vias 2 -> 0
- net RowK5: track 238.5 -> 187.9 mm
- net Row1: track 192.7 -> 143.3 mm, vias 1 -> 2
- net COM2/KS1: track 353.2 -> 306.4 mm, vias 0 -> 1
- net Row4: track 161.9 -> 115.4 mm
- net RowK6: track 189.9 -> 147.5 mm
- net COM1: track 316.5 -> 275.3 mm
- net RowK10: track 234.4 -> 193.3 mm, vias 0 -> 1
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Other:
- board size 200 x 90 mm -> 150 x 140 mm

Commit message: replace
Parts:
- moved J13 23.0 mm to (201.2, 54.8), turned to 90 degrees
- moved J14 21.1 mm to (207.1, 27.3)
- moved J3 21.1 mm to (186.8, 27.2)
- moved U4 21.1 mm to (197.2, 27.4)
- moved D12 8.03 mm to (133.6, 116.5)
- moved D14 8.03 mm to (144.2, 116.5)
- moved S11 8.03 mm to (146.4, 125.2)
- moved S9 8.03 mm to (135.6, 125.2)
- moved D10 8.03 mm to (122.9, 116.5)
- moved S7 8.03 mm to (124.8, 125.2)
- moved J12 4.96 mm to (188.2, 50.8), turned to 90 degrees
- moved J11 2.18 mm to (114.8, 32.1)
- moved R14 2.18 mm to (119.2, 32.1)
- moved R15 2.18 mm to (123.0, 32.1)
- moved S16 1.33 mm to (173.4, 125.2)
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Routing:
- net COM2/KS1: track 306.4 -> 0.00 mm, vias 1 -> 0
- net COM1: track 275.3 -> 0.00 mm, vias 1 -> 0
- net COM0: track 257.9 -> 0.00 mm, vias 1 -> 0
- net COM1/KS0: track 246.3 -> 0.00 mm
- net RowK8: track 228.1 -> 0.00 mm, vias 1 -> 0
- net RowK3: track 225.5 -> 0.00 mm, vias 2 -> 0
- net RowK7: track 200.4 -> 0.00 mm, vias 1 -> 0
- net RowK10: track 193.3 -> 0.00 mm, vias 1 -> 0
- net RowK4: track 188.3 -> 0.00 mm, vias 1 -> 0
- net RowK5: track 187.9 -> 0.00 mm, vias 1 -> 0
- net COM3/KS2: track 169.7 -> 0.00 mm, vias 1 -> 0
- net RowK9: track 168.6 -> 0.00 mm, vias 1 -> 0
- net Row0: track 160.2 -> 0.00 mm, vias 2 -> 0
- net Row3: track 159.1 -> 0.00 mm, vias 2 -> 0
- net Row2: track 158.5 -> 0.00 mm, vias 2 -> 0
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Other:
- board text added: "1"
- board text added: "2"
- board text added: "4"
- board text added: "8"
- board text added: "A"
- board text added: "A#"
- board text added: "ACC"
- board text added: "B"
- board text added: "BACK"
- board text added: "BANK"
- board text added: "C"
- board text added: "C#"
- board text added: "C2"
- board text added: "CURRENT STEP"
- board text added: "CV"
- board text added: "D"
- board text added: "D#"
- board text added: "D+3.3V"
- board text added: "D+5V"
- board text added: "DOWN"
- board text added: "E"
- board text added: "F"
- board text added: "F#"
- board text added: "FUNCTION"
- board text added: "G"
- board text added: "G#"
- board text added: "GATE"
- board text added: "GNDD"
- board text added: "HV1"
- board text added: "HV2"
- board text added: "HV3"
- board text added: "HV4"
- board text added: "I2C SCL"
- board text added: "I2C SDA"
- board text added: "LEN MAX"
- board text added: "LV1"
- board text added: "LV2"
- board text added: "LV3"
- board text added: "LV4"
- board text added: "MIDI IN"
- board text added: "NEXT"
- board text added: "NOTE"
- board text added: "ON"
- board text added: "OUTPUT"
- board text added: "PATTERN"
- board text added: "RESET"
- board text added: "RUN/STOP"
- board text added: "SLIDE"
- board text added: "SyOut"
- board text added: "TB-SEQ HT16K33 SeqBox prototype 2024/8/7"
- board text added: "TEMPO"
- board text added: "TIE"
- board text added: "TRACK"
- board text added: "UP"
- board text added: "VCC"
- board text added: "WRITE"

Commit message: HT16K33Panel DRC gaber
Parts:
- added D37: LED, LED_THT:LED_D3.0mm, F.Cu at (101.0, 42.7)
- added D38: LED, LED_THT:LED_D3.0mm, F.Cu at (105.7, 42.7)
- added D39: LED, LED_THT:LED_D3.0mm, F.Cu at (110.2, 42.8)
- added J16: Conn_01x03_Pin, Connector_PinSocket_2.54mm:PinSocket_1x03_P2.54mm_Vertical, F.Cu at (179.2, 59.0)
- added J17: Conn_01x03_Socket, Connector_PinSocket_2.54mm:PinSocket_1x03_P2.54mm_Vertical, F.Cu at (104.2, 56.8)
- added R21: 1K, Resistor_THT:R_Axial_DIN0204_L3.6mm_D1.6mm_P2.54mm_Vertical, F.Cu at (104.0, 50.9)
- added R22: 1K, Resistor_THT:R_Axial_DIN0204_L3.6mm_D1.6mm_P2.54mm_Vertical, F.Cu at (106.8, 50.9)
- added R23: 1K, Resistor_THT:R_Axial_DIN0204_L3.6mm_D1.6mm_P2.54mm_Vertical, F.Cu at (109.5, 51.0)
- moved U3 3.80 mm to (117.0, 46.5)
- moved R14 2.78 mm to (121.5, 30.5)
- moved R15 2.78 mm to (125.2, 30.5)
- moved J11 2.78 mm to (117.0, 30.5)
- moved C3 2.25 mm to (95.3, 53.1)
- moved D36 2.25 mm to (94.3, 40.1)
- moved J1 2.25 mm to (82.5, 33.3)
- moved J15 2.25 mm to (81.5, 52.8)
- moved R19 2.25 mm to (80.8, 44.8)
- moved R20 2.25 mm to (80.5, 48.6)
- moved U8 2.25 mm to (93.0, 46.6)
Routing:
- net COM2/KS1: track 0.00 -> 334.1 mm
- net COM1: track 0.00 -> 300.1 mm, vias 0 -> 2
- net COM0: track 0.00 -> 264.6 mm, vias 0 -> 1
- net RowK3: track 0.00 -> 234.8 mm, vias 0 -> 1
- net RowK8: track 0.00 -> 227.9 mm, vias 0 -> 1
- net COM1/KS0: track 0.00 -> 224.6 mm, vias 0 -> 1
- net RowK10: track 0.00 -> 220.7 mm
- net RowK7: track 0.00 -> 200.9 mm, vias 0 -> 1
- net RowK4: track 0.00 -> 185.0 mm, vias 0 -> 2
- net COM3/KS2: track 0.00 -> 176.8 mm
- net RowK9: track 0.00 -> 173.6 mm, vias 0 -> 1
- net RowK5: track 0.00 -> 171.3 mm, vias 0 -> 2
- net Row0: track 0.00 -> 162.6 mm, vias 0 -> 2
- net Row3: track 0.00 -> 160.5 mm, vias 0 -> 2
- net Row15: track 0.00 -> 160.1 mm, vias 0 -> 1
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Other:
- board text added: "RUN STOP"
- board text removed: "RUN/STOP"
