File: TBSEQ_Board_V1/HT16K33Panel/HT16K33Panel/Jack.kicad_sch (KiCad schematic)
At the start: 2 parts, among them J12 Conn_01x08_Pin, J13 Conn_01x02_Pin

Commit message: HT16K33Panel DRC gaber
Parts:
- added D37, D38, D39: LED, LED_THT:LED_D3.0mm, symbol Device:LED
- added J17: Conn_01x03_Socket, Connector_PinSocket_2.54mm:PinSocket_1x03_P2.54mm_Vertical, symbol Connector:Conn_01x03_Socket
- added R21, R22, R23: 1K, Resistor_THT:R_Axial_DIN0204_L3.6mm_D1.6mm_P2.54mm_Vertical, symbol Device:R
Connections:
- net GNDD: now also D37.1 (K), D38.1 (K), D39.1 (K)
- new net: J17.1 (Pin_1), R21.1
- new net: J17.2 (Pin_2), R22.1
- new net: J17.3 (Pin_3), R23.1
- new net: D37.2 (A), R21.2
- new net: D39.2 (A), R23.2
- new net: D38.2 (A), R22.2
