File: TBSEQ_Board_V1/HT16K33Panel/HT16K33Panel/MIDI_RX.kicad_sch (KiCad schematic)
At the start: 7 parts, among them J1 KDJ03-5, J15 Conn_01x03_Pin, U8 TLP2304_TPR,E

Commit message: HT16K33
MIDI RX動作確認済
Other:
- note added: "Vcc=5Vで動作確認済(Vcc=3.3Vだと動作できない事も確認した)"
