File: TBSEQ_Board_V1/analog_separate/Interface.kicad_sch (KiCad schematic)
At the start: 50 parts, among them IC11 AN6562, IC12 4066, J10 Conn_01x03_Pin, J2 Conn_01x05_Pin, J7 Conn_01x03_Pin, J8 Conn_01x02_Pin, J9 Conn_01x01_Pin, Q29 NPN, Q30 NPN, Q35 NPN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

Commit message: replace
Parts:
- removed J10: Conn_01x03_Pin, Connector_PinHeader_2.54mm:PinHeader_1x03_P2.54mm_Vertical, symbol Connector:Conn_01x03_Pin
- C55, C72: footprint Capacitor_THT:CP_Radial_D6.3mm_P2.50mm -> Capacitor_THT:CP_Radial_D4.0mm_P2.00mm
- C62: footprint Capacitor_THT:CP_Radial_D6.3mm_P2.50mm -> Capacitor_THT:CP_Radial_D5.0mm_P2.00mm
Connections:
- net A+CV: now also IC12.2; no longer IC12.8
- net A+ENV.MOD: now also IC12.9; no longer IC12.1
- net A+VCO_CV: now also IC12.3; no longer IC12.11
- net at Q30.2 (C), R93.1: now also IC12.13; no longer IC12.6
- net at Q29.2 (C), R91.1, R92.1: now also IC12.5; no longer IC12.12
- net at Q35.2 (C), R139.2: now also IC12.12, IC12.6; no longer IC12.13, IC12.5
- net at D28.2 (A), VR6.2 (WIPER), VR6.3 (CW): now also IC12.10; no longer IC12.4
- net at R138.1, VR6.1 (CCW): now also IC12.11; no longer IC12.3
- net at VR7.1 (CCW): now also IC12.8; no longer IC12.2
- new net: C35.1, IC12.1, IC12.4
Other:
- note removed: "PowerConnect"
