File: TBSEQ_Board_V1/analog_separate/VCA.kicad_sch (KiCad schematic)
At the start: 34 parts, among them IC15 CA3080A, K1 SJ-63072J, Q31 PNP, Q32 NPN

Commit message: replace
Parts:
- added unit 3 of VCA_IC_1
- C37, VCA_C_1: footprint Capacitor_THT:CP_Radial_D6.3mm_P2.50mm -> Capacitor_THT:CP_Radial_D4.0mm_P2.00mm
- C42: footprint Capacitor_THT:CP_Radial_D6.3mm_P2.50mm -> Capacitor_THT:CP_Radial_D5.0mm_P2.00mm
- D27, D35, D36: footprint Diode_THT:D_DO-15_P10.16mm_Horizontal -> Diode_THT:D_A-405_P2.54mm_Vertical_AnodeUp
- VCA_IC_1: footprint (none) -> Package_DIP:DIP-8_W7.62mm
Connections:
- net A+12V: now also VCA_IC_1.8 (V+)
- net GNDA: now also VCA_IC_1.4 (V-)

Commit message: fix
Parts:
- removed K1: SJ-63072J, SamacSys_Parts:SJ63072J, symbol SamacSys_Parts:SJ-63072J
- added J4: Conn_01x02_Pin, Connector_PinHeader_2.54mm:PinHeader_1x02_P2.54mm_Vertical, symbol Connector:Conn_01x02_Pin
Connections:
- net GNDA: now also J4.2 (Pin_2)
- net A+LineOut: now reaches VR8.3 (CW)
- net A+LineOut: now also J4.1 (Pin_1)
- no-connect marks 3 -> 1
Other:
- note added: "toJackBorad"
