File: TBSEQ_Board_V1/analog_separate/VCO.kicad_sch (KiCad schematic)
At the start: 32 parts, among them IC11_1 AN6562, IC11_2 AN6562, J11 Conn_01x01_Pin, J12 Conn_01x03_Pin, J13 Conn_01x01_Pin, Q24 NPN, Q25 NPN, Q26 HN4C06J-BL_6P DIP, Q27 PNP, Q28 NJFET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

Commit message: replace
Parts:
- removed J11: Conn_01x01_Pin, Connector_PinHeader_2.54mm:PinHeader_1x01_P2.54mm_Vertical, symbol Connector:Conn_01x01_Pin
- removed J12: Conn_01x03_Pin, Connector_PinHeader_2.54mm:PinHeader_1x03_P2.54mm_Vertical, symbol Connector:Conn_01x03_Pin
- removed VR_EX1: 10K(A), SamacSys_Parts:PTV1113420AA103, symbol SamacSys_Parts:PTV111-3420A-A103
- added SW1: 2MS1T1B4VS2QES, SamacSys_Parts:2MS1T1B4VS2QES, symbol SamacSys_Parts:2MS1T1B4VS2QES
- C11: footprint Capacitor_THT:CP_Radial_D6.3mm_P2.50mm -> Capacitor_THT:CP_Radial_D5.0mm_P2.00mm
- Q26: footprint SamacSys_Parts:HN4C06JBLTE85LF -> Package_DIP:DIP-6_W7.62mm
- renumbered IC11_2 to IC11_1
Connections:
- net A+VCO_SAW: now also SW1.3
- net A+VCO_SQU: now also SW1.1
- net GNDA: now also SW1.MH1, SW1.MH2
- net A+VCO_MIX renamed A+VCO_WAVE
- net A+VCO_WAVE: now also SW1.2 (2_Comm)
- no-connect marks 2 -> 1
Other:
- note removed: "PowerConnect"
- note removed: "WAVE MIX"
- note removed: "fromInterface"

Commit message: fix
Parts:
- added R100_1: 1K(TEMPCO), Resistor_THT:R_Axial_DIN0207_L6.3mm_D2.5mm_P2.54mm_Vertical, symbol Device:R
Connections:
- net A+5.333V: now also R100_1.2
- net at Q26.3 (B2), R100.1, R106.1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: now also R100_1.1
