File: TBSEQ_Board_V1/analog_separate/analog_separate.kicad_pcb (KiCad board)
At the start: 2 copper layers, 55 parts, among them IC11 AN6562, IC12 4066, J1 Conn_01x03_Pin, J10 Conn_01x03_Pin, J2 Conn_01x05_Pin, J3 Conn_01x03_Pin, J4 Conn_01x03_Pin, J5 Conn_01x03_Pin, J6 Conn_01x03_Pin, J7 Conn_01x03_Pin, J8 Conn_01x02_Pin, J9 Conn_01x01_Pin, Q29 NPN, Q30 NPN, Q35 NPN, Q36 PNP, Q37 NPN, Q38 PNP, Q39 NJFET, Q40 NPN, Q41 NPN

Commit message: replace
Parts:
- removed J10, J4, J5, J6: Conn_01x03_Pin, Connector_PinHeader_2.54mm:PinHeader_1x03_P2.54mm_Vertical
- added C10: 0.01uF, Capacitor_THT:C_Rect_L7.2mm_W2.5mm_P5.00mm_FKS2_FKP2_MKS2_MKP2, F.Cu at (47.8, 86.2)
- added C11: 1uF/50V, Capacitor_THT:CP_Radial_D5.0mm_P2.00mm, F.Cu at (57.1, 88.5)
- added C13: 1uF/50V, Capacitor_THT:CP_Radial_D5.0mm_P2.00mm, F.Cu at (147.8, 59.7)
- added C14: 1uF/50V, Capacitor_THT:CP_Radial_D5.0mm_P2.00mm, F.Cu at (148.6, 84.7)
- added C15: 1uF/50V, Capacitor_THT:CP_Radial_D5.0mm_P2.00mm, F.Cu at (112.3, 78.7)
- added C16: 10uF/16V, Capacitor_THT:CP_Radial_D4.0mm_P2.00mm, F.Cu at (68.1, 69.5)
- added C17: 1uF/50V, Capacitor_THT:CP_Radial_D5.0mm_P2.00mm, F.Cu at (74.6, 58.2)
- added C18: 0.018uF, Capacitor_THT:C_Rect_L7.2mm_W2.5mm_P5.00mm_FKS2_FKP2_MKS2_MKP2, F.Cu at (94.3, 65.2)
- added C19: 0.033uF, Capacitor_THT:C_Rect_L7.2mm_W2.5mm_P5.00mm_FKS2_FKP2_MKS2_MKP2, F.Cu at (102.3, 65.2)
- added C20: 0.01uF, Capacitor_THT:C_Rect_L7.2mm_W2.5mm_P5.00mm_FKS2_FKP2_MKS2_MKP2, F.Cu at (163.2, 70.0)
- added C21: 0.01uF, Capacitor_THT:C_Rect_L7.2mm_W2.5mm_P5.00mm_FKS2_FKP2_MKS2_MKP2, F.Cu at (163.2, 74.0)
- added C22: 1uF/50V, Capacitor_THT:CP_Radial_D5.0mm_P2.00mm, F.Cu at (112.3, 87.5)
- added C23: 1uF/50V, Capacitor_THT:CP_Radial_D5.0mm_P2.00mm, F.Cu at (96.6, 77.7)
- added C24: 0.033uF, Capacitor_THT:C_Rect_L7.2mm_W2.5mm_P5.00mm_FKS2_FKP2_MKS2_MKP2, F.Cu at (110.3, 65.1)
- added C25: 0.1uF, Capacitor_THT:C_Rect_L7.2mm_W2.5mm_P5.00mm_FKS2_FKP2_MKS2_MKP2, F.Cu at (120.5, 71.6)
- added C26: 0.033uF, Capacitor_THT:C_Rect_L7.2mm_W2.5mm_P5.00mm_FKS2_FKP2_MKS2_MKP2, F.Cu at (118.5, 61.8)
- added C27: 0.1uF, Capacitor_THT:C_Rect_L7.2mm_W2.5mm_P5.00mm_FKS2_FKP2_MKS2_MKP2, F.Cu at (129.0, 71.6)
- added C28: 47uF/16V, Capacitor_THT:CP_Radial_D4.0mm_P2.00mm, F.Cu at (141.0, 65.5)
- added C29: 1uF/50V, Capacitor_THT:CP_Radial_D5.0mm_P2.00mm, F.Cu at (132.1, 86.5)
- added C30: 10uF/16V, Capacitor_THT:CP_Radial_D4.0mm_P2.00mm, F.Cu at (135.0, 65.5)
- added C33: 0.01uF, Capacitor_THT:C_Rect_L7.2mm_W2.5mm_P5.00mm_FKS2_FKP2_MKS2_MKP2, F.Cu at (47.7, 74.7)
- added C34: 0.001uF, Capacitor_THT:C_Rect_L7.2mm_W2.5mm_P5.00mm_FKS2_FKP2_MKS2_MKP2, F.Cu at (31.9, 77.5)
- added C36: 0.033uF, Capacitor_THT:C_Rect_L7.2mm_W2.5mm_P5.00mm_FKS2_FKP2_MKS2_MKP2, F.Cu at (203.5, 85.0)
- added C37: 10uF/16V, Capacitor_THT:CP_Radial_D4.0mm_P2.00mm, F.Cu at (164.5, 64.2)
- added C41: 0.1uF, Capacitor_THT:C_Rect_L7.2mm_W2.5mm_P5.00mm_FKS2_FKP2_MKS2_MKP2, F.Cu at (169.0, 85.2)
- added C42: 1uF/50V, Capacitor_THT:CP_Radial_D5.0mm_P2.00mm, F.Cu at (191.2, 87.5)
- added D24: D, Diode_THT:D_A-405_P2.54mm_Vertical_AnodeUp, F.Cu at (147.3, 69.5)
- added D25: D, Diode_THT:D_A-405_P2.54mm_Vertical_AnodeUp, F.Cu at (53.3, 58.8)
- added D27: D, Diode_THT:D_A-405_P2.54mm_Vertical_AnodeUp, F.Cu at (204.4, 89.3)
- added D35: D, Diode_THT:D_A-405_P2.54mm_Vertical_AnodeUp, F.Cu at (163.5, 80.2)
- added D36: D, Diode_THT:D_A-405_P2.54mm_Vertical_AnodeUp, F.Cu at (163.5, 85.2)
- added IC11_1: AN6562, Package_DIP:DIP-8_W7.62mm, F.Cu at (35.7, 72.9)
- added IC15: CA3080A, Package_DIP:DIP-8_W7.62mm, F.Cu at (179.2, 66.0)
- added J13: Conn_01x01_Pin, Connector_PinHeader_2.54mm:PinHeader_1x01_P2.54mm_Vertical, F.Cu at (60.7, 59.0)
- added K1: SJ-63072J, SamacSys_Parts:SJ63072J, F.Cu at (235.6, 36.2)
- added Q10: PNP, Package_TO_SOT_THT:TO-92_Inline, F.Cu at (83.3, 86.5)
- added Q11: NPN, Package_TO_SOT_THT:TO-92_Inline, F.Cu at (80.8, 81.5)
- added Q12: HN4C06J-BL_6P DIP, Package_DIP:DIP-6_W7.62mm, F.Cu at (80.8, 66.9)
- added Q13: NPN, Package_TO_SOT_THT:TO-92_Inline, F.Cu at (95.3, 60.3)
- added Q14: NPN, Package_TO_SOT_THT:TO-92_Inline, F.Cu at (103.0, 60.3)
- added Q15: NPN, Package_TO_SOT_THT:TO-92_Inline, F.Cu at (95.3, 70.1)
- added Q16: NPN, Package_TO_SOT_THT:TO-92_Inline, F.Cu at (110.8, 60.2)
- added Q17: NPN, Package_TO_SOT_THT:TO-92_Inline, F.Cu at (103.8, 70.1)
- added Q18: NPN, Package_TO_SOT_THT:TO-92_Inline, F.Cu at (103.8, 78.0)
- added Q19: NPN, Package_TO_SOT_THT:TO-92_Inline, F.Cu at (144.9, 84.6)
- added Q20: NPN, Package_TO_SOT_THT:TO-92_Inline, F.Cu at (120.3, 85.5)
- added Q21: HN4C06J-BL_6P DIP, Package_DIP:DIP-6_W7.62mm, F.Cu at (131.6, 77.2)
- added Q22: DMMT3906_6P DIP, Package_DIP:DIP-6_W7.62mm, F.Cu at (128.6, 59.5)
- added Q23: NPN, Package_TO_SOT_THT:TO-92_Inline, F.Cu at (111.0, 70.0)
- added Q24: NPN, Package_TO_SOT_THT:TO-92_Inline, F.Cu at (53.3, 63.6)
- added Q25: NPN, Package_TO_SOT_THT:TO-92_Inline, F.Cu at (45.0, 64.5)
- added Q26: HN4C06J-BL_6P DIP, Package_DIP:DIP-6_W7.62mm, F.Cu at (34.2, 59.2)
- added Q27: PNP, Package_TO_SOT_THT:TO-92_Inline, F.Cu at (45.0, 59.6)
- added Q28: NJFET, Package_TO_SOT_THT:TO-92_Inline, F.Cu at (51.2, 71.3)
- added Q31: PNP, Package_TO_SOT_THT:TO-92_Inline, F.Cu at (182.5, 80.5)
- added Q32: NPN, Package_TO_SOT_THT:TO-92_Inline, F.Cu at (178.2, 88.5)
- added Q8: PNP, Package_TO_SOT_THT:TO-92_Inline, F.Cu at (59.6, 75.7)
- added Q9: PNP, Package_TO_SOT_THT:TO-92_Inline, F.Cu at (77.4, 86.5)
- added R100: 1K(TEMPCO), Resistor_THT:R_Axial_DIN0207_L6.3mm_D2.5mm_P2.54mm_Vertical, F.Cu at (29.7, 61.5)
- added R101: 10K, Resistor_THT:R_Axial_DIN0207_L6.3mm_D2.5mm_P2.54mm_Vertical, F.Cu at (56.5, 62.8)
- added R102: 100K, Resistor_THT:R_Axial_DIN0207_L6.3mm_D2.5mm_P2.54mm_Vertical, F.Cu at (32.0, 86.7)
- added R103: 220K, Resistor_THT:R_Axial_DIN0207_L6.3mm_D2.5mm_P2.54mm_Vertical, F.Cu at (32.0, 83.0)
- added R104: 2.2K, Resistor_THT:R_Axial_DIN0207_L6.3mm_D2.5mm_P2.54mm_Vertical, F.Cu at (29.7, 64.9)
- added R105: 10K, Resistor_THT:R_Axial_DIN0207_L6.3mm_D2.5mm_P2.54mm_Vertical, F.Cu at (53.5, 76.5)
- added R106: 27K, Resistor_THT:R_Axial_DIN0207_L6.3mm_D2.5mm_P2.54mm_Vertical, F.Cu at (26.2, 67.0)
- added R108: 2.2K, Resistor_THT:R_Axial_DIN0207_L6.3mm_D2.5mm_P2.54mm_Vertical, F.Cu at (119.9, 90.0)
- added R109: 10K, Resistor_THT:R_Axial_DIN0207_L6.3mm_D2.5mm_P2.54mm_Vertical, F.Cu at (123.1, 90.0)
- added R110: 22K, Resistor_THT:R_Axial_DIN0207_L6.3mm_D2.5mm_P2.54mm_Vertical, F.Cu at (144.6, 80.2)
- added R111: 22K, Resistor_THT:R_Axial_DIN0207_L6.3mm_D2.5mm_P2.54mm_Vertical, F.Cu at (144.6, 77.0)
- added R112: 10K, Resistor_THT:R_Axial_DIN0207_L6.3mm_D2.5mm_P2.54mm_Vertical, F.Cu at (126.3, 84.2)
- added R113: 100K, Resistor_THT:R_Axial_DIN0207_L6.3mm_D2.5mm_P2.54mm_Vertical, F.Cu at (126.3, 80.5)
- added R114: 100K, Resistor_THT:R_Axial_DIN0207_L6.3mm_D2.5mm_P2.54mm_Vertical, F.Cu at (122.1, 80.5)
- added R115: 10K, Resistor_THT:R_Axial_DIN0207_L6.3mm_D2.5mm_P2.54mm_Vertical, F.Cu at (137.3, 60.0)
- added R116: 10K, Resistor_THT:R_Axial_DIN0207_L6.3mm_D2.5mm_P2.54mm_Vertical, F.Cu at (137.4, 88.7)
- added R118: 100K, Resistor_THT:R_Axial_DIN0207_L6.3mm_D2.5mm_P2.54mm_Vertical, F.Cu at (26.2, 59.4)
- added R119: 47K, Resistor_THT:R_Axial_DIN0207_L6.3mm_D2.5mm_P2.54mm_Vertical, F.Cu at (197.7, 85.0)
- added R120: 22K, Resistor_THT:R_Axial_DIN0207_L6.3mm_D2.5mm_P2.54mm_Vertical, F.Cu at (197.7, 89.0)
- added R121: 220K, Resistor_THT:R_Axial_DIN0207_L6.3mm_D2.5mm_P2.54mm_Vertical, F.Cu at (172.0, 70.2)
- added R122: 100K, Resistor_THT:R_Axial_DIN0207_L6.3mm_D2.5mm_P2.54mm_Vertical, F.Cu at (172.0, 74.2)
- added R123: 1.5M, Resistor_THT:R_Axial_DIN0207_L6.3mm_D2.5mm_P2.54mm_Vertical, F.Cu at (184.7, 85.5)
- added R124: 2.2K, Resistor_THT:R_Axial_DIN0207_L6.3mm_D2.5mm_P2.54mm_Vertical, F.Cu at (171.5, 61.7)
- added R125: 2.2K, Resistor_THT:R_Axial_DIN0207_L6.3mm_D2.5mm_P2.54mm_Vertical, F.Cu at (171.5, 65.8)
- added R126: 2.2K, Resistor_THT:R_Axial_DIN0207_L6.3mm_D2.5mm_P2.54mm_Vertical, F.Cu at (164.7, 59.2)
- added R130: 100, Resistor_THT:R_Axial_DIN0207_L6.3mm_D2.5mm_P2.54mm_Vertical, F.Cu at (169.2, 89.2)
- added R131: 220K, Resistor_THT:R_Axial_DIN0207_L6.3mm_D2.5mm_P2.54mm_Vertical, F.Cu at (175.4, 80.0)
- added R132: 100, Resistor_THT:R_Axial_DIN0207_L6.3mm_D2.5mm_P2.54mm_Vertical, F.Cu at (184.7, 90.5)
- added R133: 2.2K, Resistor_THT:R_Axial_DIN0207_L6.3mm_D2.5mm_P2.54mm_Vertical, F.Cu at (169.7, 80.2)
- added R134: 22K, Resistor_THT:R_Axial_DIN0207_L6.3mm_D2.5mm_P2.54mm_Vertical, F.Cu at (163.4, 89.2)
- added R34: 10K, Resistor_THT:R_Axial_DIN0207_L6.3mm_D2.5mm_P2.54mm_Vertical, F.Cu at (51.6, 86.9)
- added R35: 100K, Resistor_THT:R_Axial_DIN0207_L6.3mm_D2.5mm_P2.54mm_Vertical, F.Cu at (51.6, 83.5)
- added R36: 10K, Resistor_THT:R_Axial_DIN0207_L6.3mm_D2.5mm_P2.54mm_Vertical, F.Cu at (59.6, 80.7)
- added R45: 22K, Resistor_THT:R_Axial_DIN0207_L6.3mm_D2.5mm_P2.54mm_Vertical, F.Cu at (55.8, 82.7)
- added R46: 47K, Resistor_THT:R_Axial_DIN0207_L6.3mm_D2.5mm_P2.54mm_Vertical, F.Cu at (149.3, 65.7)
- added R47: 10K, Resistor_THT:R_Axial_DIN0207_L6.3mm_D2.5mm_P2.54mm_Vertical, F.Cu at (83.1, 59.7)
- added R61: 10K, Resistor_THT:R_Axial_DIN0207_L6.3mm_D2.5mm_P2.54mm_Vertical, F.Cu at (89.1, 59.5)
- added R62: 220K, Resistor_THT:R_Axial_DIN0207_L6.3mm_D2.5mm_P2.54mm_Vertical, F.Cu at (67.0, 59.2)
- added R63: 220K, Resistor_THT:R_Axial_DIN0207_L6.3mm_D2.5mm_P2.54mm_Vertical, F.Cu at (88.9, 87.5)
- added R64: 10K, Resistor_THT:R_Axial_DIN0207_L6.3mm_D2.5mm_P2.54mm_Vertical, F.Cu at (73.3, 80.2)
- added R65: 10K, Resistor_THT:R_Axial_DIN0207_L6.3mm_D2.5mm_P2.54mm_Vertical, F.Cu at (73.3, 77.0)
- added R66: 100K, Resistor_THT:R_Axial_DIN0207_L6.3mm_D2.5mm_P2.54mm_Vertical, F.Cu at (107.0, 89.5)
- added R67: 2.2K, Resistor_THT:R_Axial_DIN0207_L6.3mm_D2.5mm_P2.54mm_Vertical, F.Cu at (111.0, 82.5)
- added R68: 2.2K, Resistor_THT:R_Axial_DIN0207_L6.3mm_D2.5mm_P2.54mm_Vertical, F.Cu at (69.3, 65.2)
- added R69: 2.2K, Resistor_THT:R_Axial_DIN0207_L6.3mm_D2.5mm_P2.54mm_Vertical, F.Cu at (73.3, 73.7)
- added R70: 2.2K, Resistor_THT:R_Axial_DIN0207_L6.3mm_D2.5mm_P2.54mm_Vertical, F.Cu at (75.4, 65.2)
- added R71: 2.2K, Resistor_THT:R_Axial_DIN0207_L6.3mm_D2.5mm_P2.54mm_Vertical, F.Cu at (83.3, 92.2)
- added R72: 100K, Resistor_THT:R_Axial_DIN0207_L6.3mm_D2.5mm_P2.54mm_Vertical, F.Cu at (88.8, 83.7)
- added R73: 100K, Resistor_THT:R_Axial_DIN0207_L6.3mm_D2.5mm_P2.54mm_Vertical, F.Cu at (86.8, 80.0)
- added R94: 10K, Resistor_THT:R_Axial_DIN0207_L6.3mm_D2.5mm_P2.54mm_Vertical, F.Cu at (103.5, 87.5)
- added R95: 100, Resistor_THT:R_Axial_DIN0207_L6.3mm_D2.5mm_P2.54mm_Vertical, F.Cu at (143.1, 59.8)
- added R96: 10K, Resistor_THT:R_Axial_DIN0207_L6.3mm_D2.5mm_P2.54mm_Vertical, F.Cu at (142.6, 89.5)
- added R97: 10K, Resistor_THT:R_Axial_DIN0207_L6.3mm_D2.5mm_P2.54mm_Vertical, F.Cu at (88.9, 76.2)
- added R98: 2.2K, Resistor_THT:R_Axial_DIN0207_L6.3mm_D2.5mm_P2.54mm_Vertical, F.Cu at (73.3, 70.5)
- added R99: 100K, Resistor_THT:R_Axial_DIN0207_L6.3mm_D2.5mm_P2.54mm_Vertical, F.Cu at (104.3, 82.5)
- added SW1: 2MS1T1B4VS2QES, SamacSys_Parts:2MS1T1B4VS2QES, F.Cu at (36.7, 43.0)
- added TM3: 500K, SamacSys_Parts:3296W1502A, F.Cu at (96.8, 90.2)
- added TM4: 50K, SamacSys_Parts:3296W1502A, F.Cu at (37.5, 87.7)
- added TM5: 5K, SamacSys_Parts:3296W1502A, F.Cu at (25.5, 74.5)
- added VCA_C_1: 10uF/16V, Capacitor_THT:CP_Radial_D4.0mm_P2.00mm, F.Cu at (201.5, 59.9)
- added VCA_IC_1: Opamp_Dual, Package_DIP:DIP-8_W7.62mm, F.Cu at (197.9, 66.5)
- added VCA_R1: 10K, Resistor_THT:R_Axial_DIN0207_L6.3mm_D2.5mm_P2.54mm_Vertical, F.Cu at (194.0, 74.2)
- added VCA_R2: 100, Resistor_THT:R_Axial_DIN0207_L6.3mm_D2.5mm_P2.54mm_Vertical, F.Cu at (196.5, 62.7)
- added VCA_R3: 100K, Resistor_THT:R_Axial_DIN0207_L6.3mm_D2.5mm_P2.54mm_Vertical, F.Cu at (194.2, 66.4)
- added VCA_R4: 100K, Resistor_THT:R_Axial_DIN0207_L6.3mm_D2.5mm_P2.54mm_Vertical, F.Cu at (207.5, 59.4)
- added VCA_R5: 47K, Resistor_THT:R_Axial_DIN0207_L6.3mm_D2.5mm_P2.54mm_Vertical, F.Cu at (189.8, 79.8)
- added VR2: 50K(B), SamacSys_Parts:PTV1113420AA103, F.Cu at (51.9, 49.7)
- added VR3: 50K(A), SamacSys_Parts:PTV1113420AA103, F.Cu at (77.0, 49.9)
- added VR4: 50K(B)2連, SamacSys_Parts:PTV1124420AA504, F.Cu at (102.8, 49.8)
- added VR5: 50K(A), SamacSys_Parts:PTV1113420AA103, F.Cu at (125.3, 49.9)
- added VR8: 10K(B), SamacSys_Parts:PTV1113420AA103, F.Cu at (193.3, 50.7)
- C55, C72: footprint Capacitor_THT:CP_Radial_D6.3mm_P2.50mm -> Capacitor_THT:CP_Radial_D4.0mm_P2.00mm
- C62: footprint Capacitor_THT:CP_Radial_D6.3mm_P2.50mm -> Capacitor_THT:CP_Radial_D5.0mm_P2.00mm
- J3: value Conn_01x03_Pin -> Conn_01x02_Pin; footprint Connector_PinHeader_2.54mm:PinHeader_1x03_P2.54mm_Vertical -> Connector_PinHeader_2.54mm:PinHeader_1x02_P2.54mm_Vertical
- moved J9 214.0 mm to (25.2, 106.4)
- moved D31 196.7 mm to (29.2, 106.4), turned to -90 degrees
- moved D32 196.7 mm to (29.2, 111.9), turned to -90 degrees
- moved IC11 176.8 mm to (35.9, 106.1)
- moved R107 176.0 mm to (33.0, 108.7)
- moved R92 148.5 mm to (50.1, 109.0), turned to 180 degrees
- moved R93 148.5 mm to (50.1, 112.7), turned to 180 degrees
- moved R91 143.2 mm to (55.6, 112.7), turned to 180 degrees
- moved Q30 137.8 mm to (53.3, 109.0)
- moved R117 132.9 mm to (83.9, 104.5), turned to 180 degrees
- moved Q29 132.8 mm to (58.8, 109.0)
- moved C35 129.0 mm to (107.3, 105.2), turned to 90 degrees
- moved D26 128.3 mm to (87.8, 104.5)
- moved R59 123.7 mm to (61.1, 112.7), turned to 180 degrees
- moved D29 121.6 mm to (94.0, 104.5)
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Connections:
- IC12 pad 1: A+ENV.MOD -> Net-(C35-Pad1)
- IC12 pad 10: Net-(C35-Pad1) -> Net-(D28-A)
- IC12 pad 11: A+VCO_CV -> Net-(VR6-CCW)
- IC12 pad 12: Net-(Q29-C) -> Net-(Q35-C)
- IC12 pad 13: Net-(Q35-C) -> Net-(Q30-C)
- IC12 pad 2: Net-(VR7-CCW) -> A+CV
- IC12 pad 3: Net-(VR6-CCW) -> A+VCO_CV
- IC12 pad 4: Net-(D28-A) -> Net-(C35-Pad1)
- IC12 pad 5: Net-(Q35-C) -> Net-(Q29-C)
- IC12 pad 6: Net-(Q30-C) -> Net-(Q35-C)
- IC12 pad 8: A+CV -> Net-(VR7-CCW)
- IC12 pad 9: Net-(C35-Pad1) -> A+ENV.MOD
- J3 pad 1: A+12V -> A+VCA_Signal
- J3 pad 2: A+5.333V -> A+VCA_Resonance
Routing:
- net A+12V: track 24.4 -> 216.4 mm
- net A+5.333V: track 24.4 -> 201.7 mm, vias 0 -> 1
- net A+VCO_CV: track 0.00 -> 106.8 mm, vias 0 -> 4
- net A+CV: track 0.00 -> 88.2 mm, vias 0 -> 2
- net Net-(Q35-C): track 0.00 -> 58.5 mm, vias 0 -> 1
- net D+GATE: track 0.00 -> 37.5 mm
- net A+ENV_Trig: track 0.00 -> 34.0 mm
- net D-ACC: track 0.00 -> 28.0 mm, vias 0 -> 2
- net Net-(D28-A): track 0.00 -> 25.0 mm
- net Net-(Q41-B): track 0.00 -> 20.5 mm
- net Net-(Q29-C): track 0.00 -> 17.4 mm
- net Net-(D26-A): track 0.00 -> 17.0 mm, vias 0 -> 2
- net Net-(C35-Pad1): track 0.00 -> 15.2 mm
- net Net-(Q36-B): track 0.00 -> 14.3 mm
- net Net-(Q38-E): track 0.00 -> 13.7 mm
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- added copper zone on B.Cu, net GNDA
- added copper zone on F.Cu, net GNDA
Other:
- board text added: "A+12V"
- board text added: "A+5.333V"
- board text added: "CUTOFF FREQ."
- board text added: "ENV.MOD"
- board text added: "GNDA"
- board text added: "OUTPUT"
- board text added: "RESONANCE"
- board text added: "TUNING"
- board text added: "VOLUME"
- board text added: "WAVE"

Commit message: fix
Parts:
- removed K1: SJ-63072J, SamacSys_Parts:SJ63072J
- added J4: Conn_01x02_Pin, Connector_PinHeader_2.54mm:PinHeader_1x02_P2.54mm_Vertical, F.Cu at (223.0, 80.0)
- added J5: Conn_01x03_Pin, Connector_PinHeader_2.54mm:PinHeader_1x03_P2.54mm_Vertical, F.Cu at (213.9, 131.0)
- added R100_1: 1K(TEMPCO), Resistor_THT:R_Axial_DIN0207_L6.3mm_D2.5mm_P2.54mm_Vertical, F.Cu at (47.2, 76.3)
- moved R130 32.6 mm to (197.8, 105.1), turned to -90 degrees
- moved J3 31.2 mm to (170.8, 105.2), turned to 0 degrees
- moved TM5 31.0 mm to (46.0, 97.7)
- moved R134 30.6 mm to (192.3, 99.4), turned to 180 degrees
- moved R121 29.8 mm to (192.2, 92.0), turned to 180 degrees
- moved R124 29.5 mm to (192.3, 82.5), turned to 180 degrees
- moved R126 28.3 mm to (186.1, 77.8), turned to 180 degrees
- moved C22 27.5 mm to (135.5, 102.2)
- moved J9 27.0 mm to (45.5, 124.2)
- moved C54 26.9 mm to (173.6, 131.2)
- moved C55 26.9 mm to (188.8, 124.4)
- moved Q38 26.9 mm to (183.8, 128.7)
- moved J2 26.9 mm to (88.7, 130.9)
- moved R59 26.9 mm to (81.3, 130.4)
- moved R91 26.9 mm to (75.8, 130.4)
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Connections:
- VR8 pad 3: Net-(K1-TIP) -> A+LineOut
Routing:
- net A+12V: track 216.4 -> 448.7 mm
- net A+5.333V: track 201.7 -> 396.4 mm, vias 1 -> 0
- net A+ENV.MOD: track 3.48 -> 136.2 mm
- net A+VCA-Reso_ACC: track 0.00 -> 125.8 mm
- net Net-(VR6-CCW): track 0.00 -> 124.8 mm
- net A+VCA_Resonance: track 0.00 -> 108.0 mm
- net A+VCA_Signal: track 0.00 -> 97.8 mm
- net Net-(Q30-C): track 7.51 -> 77.7 mm
- net Net-(VR7-CCW): track 0.00 -> 69.9 mm
- net Net-(Q29-C): track 17.4 -> 86.8 mm
- net Net-(D28-A): track 25.0 -> 90.8 mm
- net A+VCO_SAW: track 0.00 -> 64.9 mm, vias 0 -> 1
- net Net-(VR4-CCW_2): track 0.00 -> 58.1 mm
- net A+VCO_SQU: track 0.00 -> 56.0 mm
- net Net-(VR5-WIPER): track 0.00 -> 55.3 mm
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Other:
- board outline added: 200 x 100 mm
- board text added: "A+ENV.MOD"
- board text added: "A+VCA Reso_ACC"
- board text added: "A+VCA_Env"
- board text added: "A+VCA_Resonance"
- board text added: "A+VCA_Signal"
- board text added: "A+VCA_Trig"
- board text added: "A+VCO_CV"
- board text added: "A+VCO_WAVE"
- board text added: "FREQ"
- board text added: "LineOut"
- board text added: "TB-SEQ 303Borad 2024/8/15"
- board text added: "TUNE"
- board text added: "WIDTH"
- board text removed: "OUTPUT"

Commit message: analog_separate fix
実装してバグを修正
・VR6以外のボリュームの左右が逆なのを修正
・デュアルトランジスタをHN1C01FU-GRに変更
・VCA CA3080後の出力段のバイアス/増幅率等の設計ミスを修正
・入力信号のシルク位置が間違っているので修正
⇒それ以外は正常動作を確認済
Parts:
- added VCA_C_2: 10uF/16V, Capacitor_THT:CP_Radial_D4.0mm_P2.00mm, F.Cu at (201.2, 71.9)
- added VCA_R6: 100K, Resistor_THT:R_Axial_DIN0207_L6.3mm_D2.5mm_P2.54mm_Vertical, F.Cu at (209.2, 75.5)
- added VCA_R7: 100K, Resistor_THT:R_Axial_DIN0207_L6.3mm_D2.5mm_P2.54mm_Vertical, F.Cu at (209.2, 80.8)
- Q12, Q21, Q26: value HN4C06J-BL_6P DIP -> HN1C01FU-GR,LF_6P DIP
- Q22: value DMMT3906_6P DIP -> HN1C01FU-GR,LF_6P DIP
- VCA_R3: value 100K -> 47K
- moved J4 7.39 mm to (230.3, 78.9)
- moved VCA_IC_1 6.38 mm to (218.0, 78.1)
- moved VCA_R1 6.38 mm to (214.4, 83.5)
- moved VCA_R3 6.38 mm to (214.4, 78.1)
- moved VCA_C_1 6.21 mm to (220.2, 72.1)
- moved VCA_R4 5.90 mm to (226.2, 72.1)
- moved VCA_R2 5.84 mm to (216.0, 73.2)
- moved Q12 1.99 mm to (102.5, 79.9)
- moved Q21 1.24 mm to (151.4, 91.4)
- moved Q22 1.05 mm to (149.3, 73.3)
- moved Q26 0.75 mm to (55.4, 73.3)
Connections:
- C13 pad 1: Net-(VR4-CCW_2) -> Net-(VR4-CW_2)
- C30 pad 1: Net-(Q22-B12) -> Net-(Q22-B1)
- IC12 pad 8: Net-(VR7-CCW) -> Net-(VR7-CW)
- IC15 pad 6: Net-(VCA_IC_1A-+) -> Net-(IC15-Pad6)
- Q12 pad 1: Net-(Q12-B1) -> Net-(Q12-E1)
- Q12 pad 2: Net-(Q12-E) -> Net-(Q12-B1)
- Q12 pad 3: Net-(Q12-B2) -> Net-(Q12-C2)
- Q12 pad 4: Net-(Q12-C2) -> Net-(Q12-E1)
- Q12 pad 5: unconnected-(Q12-NC-Pad5) -> Net-(Q12-B2)
- Q21 pad 1: Net-(Q21-B1) -> Net-(Q20-C)
- Q21 pad 2: Net-(Q20-C) -> Net-(Q21-B1)
- Q21 pad 3: Net-(Q21-B2) -> Net-(Q19-B)
- Q21 pad 4: Net-(Q19-B) -> Net-(Q20-C)
- Q21 pad 5: unconnected-(Q21-NC-Pad5) -> Net-(Q21-B2)
- Q22 pad 2: unconnected-(Q22-NC-Pad2) -> Net-(Q22-B1)
- Q22 pad 3: Net-(Q22-E2) -> Net-(Q19-C)
- Q22 pad 4: Net-(Q19-C) -> Net-(Q22-E2)
- Q22 pad 5: Net-(Q22-B12) -> Net-(Q22-B1)
- Q26 pad 1: A+5.333V -> Net-(Q26-E1)
- Q26 pad 2: Net-(Q26-E) -> A+5.333V
- Q26 pad 3: Net-(Q26-B2) -> Net-(Q25-E)
- Q26 pad 4: Net-(Q25-E) -> Net-(Q26-E1)
- Q26 pad 5: unconnected-(Q26-NC-Pad5) -> Net-(Q26-B2)
- R104 pad 1: Net-(Q26-E) -> Net-(Q26-E1)
- R115 pad 2: Net-(Q22-B12) -> Net-(Q22-B1)
- R46 pad 1: Net-(VR4-CW_2) -> Net-(VR4-CCW_2)
- R47 pad 1: Net-(VR3-CW) -> Net-(VR3-CCW)
- R61 pad 1: Net-(VR5-CW) -> Net-(VR5-CCW)
- R69 pad 2: Net-(Q12-E) -> Net-(Q12-E1)
- VCA_C_1 pad 2: Net-(VR8-CCW) -> Net-(VR8-CW)
- VCA_IC_1 pad 6: GNDA -> A+5.333V
- VCA_R4 pad 1: Net-(VR8-CCW) -> Net-(VR8-CW)
- VR2 pad 1: A+5.333V -> GNDA
- VR2 pad 3: GNDA -> A+5.333V
- VR3 pad 1: A+12V -> Net-(VR3-CCW)
- VR3 pad 3: Net-(VR3-CW) -> A+12V
- VR4 pad A1: A+VCA_Signal -> GNDA
- VR4 pad A3: GNDA -> A+VCA_Signal
- VR5 pad 1: A+ENV.MOD -> Net-(VR5-CCW)
- VR5 pad 3: Net-(VR5-CW) -> A+ENV.MOD
- VR7 pad 1: Net-(VR7-CCW) -> GNDA
- VR7 pad 3: GNDA -> Net-(VR7-CW)
- VR8 pad 1: Net-(VR8-CCW) -> GNDA
- VR8 pad 2: Net-(VR8-CCW) -> A+LineOut
- VR8 pad 3: A+LineOut -> Net-(VR8-CW)
Routing:
- net Net-(VR7-CW): track 0.00 -> 85.1 mm, vias 0 -> 3
- net Net-(VR7-CCW): track 69.9 -> 0.00 mm
- net Net-(VR5-CW): track 44.6 -> 0.00 mm
- net Net-(VR5-CCW): track 0.00 -> 39.6 mm
- net Net-(Q22-B1): track 0.00 -> 30.2 mm, vias 0 -> 1
- net GNDA: track 21.1 -> 46.4 mm, vias 6 -> 4
- net Net-(Q12-E1): track 0.00 -> 22.0 mm
- net A+5.333V: track 396.4 -> 418.3 mm, vias 0 -> 2
- net Net-(Q26-E1): track 0.00 -> 19.2 mm
- net Net-(Q22-B12): track 15.3 -> 0.00 mm
- net Net-(VR8-CCW): track 15.0 -> 0.00 mm
- net Net-(VR3-CCW): track 0.00 -> 14.5 mm
- net Net-(VR8-CW): track 0.00 -> 13.8 mm
- net Net-(VCA_IC_1A-+): track 9.29 -> 22.4 mm
- net Net-(Q20-C): track 13.0 -> 25.9 mm, vias 0 -> 1
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Other:
- board text added: "TB-SEQ 303Borad V0.2 2024/9/23"
- board text removed: "TB-SEQ 303Borad 2024/8/15"
