File: TBSEQ_Board_V1/powersupply/powersupply/powersupply.kicad_sch (KiCad schematic)
At the start: 27 parts, among them J1 Conn_01x02_Pin, J2 DF1BZ-3P-2.5DS, J3 Barrel_Jack_Switch, J4 Conn_01x02_Pin, J5 Conn_01x02_Pin, J6 Conn_01x02_Pin, J8 DF1BZ-2P-2.5DSA, U3 L7812, U4 LM317_TO-220

Commit message: fix
Parts:
- VR1: value 3296W-1-502A -> 3296W-1-101LF
Changed lines of the file:
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@@
 			)
 		)
-		(property "Value" "3296W-1-502A"
+		(property "Value" "3296W-1-101LF"
 			(at 204.724 89.662 0)
 			(effects
