File: TBSEQ_Board_V1/analog_separate/組み立てデバッグ前/Interface.kicad_sch (KiCad schematic)
At the start: 49 parts, among them IC11 AN6562, IC12 4066, J2 Conn_01x05_Pin, J7 Conn_01x03_Pin, J8 Conn_01x02_Pin, J9 Conn_01x01_Pin, Q29 NPN, Q30 NPN, Q35 NPN, Q36 PNP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

Commit message: analog_separate fix
実装してバグを修正
・VR6以外のボリュームの左右が逆なのを修正
・デュアルトランジスタをHN1C01FU-GRに変更
・VCA CA3080後の出力段のバイアス/増幅率等の設計ミスを修正
・入力信号のシルク位置が間違っているので修正
⇒それ以外は正常動作を確認済
Connections:
- net GNDA: now also VR7.3 (CW); no longer VR7.1 (CCW)
- net at IC12.8: now also VR7.1 (CCW); no longer VR7.3 (CW)
Changed lines of the file:
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@@
 	(wire
 		(pts
+			(xy 153.67 96.52) (xy 88.9 96.52)
+		)
+		(stroke
+			(width 0)
+			(type default)
+		)
+	)
+	(wire
+		(pts
 			(xy 96.52 104.14) (xy 59.69 104.14)
 		)
@@
 	(wire
 		(pts
-			(xy 163.83 83.82) (xy 163.83 85.09)
-		)
-		(stroke
-			(width 0)
-			(type default)
-		)
-	)
-	(wire
-		(pts
 			(xy 231.14 118.11) (xy 229.87 118.11)
 		)
@@
 	(wire
 		(pts
-			(xy 62.23 132.08) (xy 69.85 132.08)
+			(xy 88.9 96.52) (xy 88.9 90.17)
 		)
 		(stroke
@@
 	(wire
 		(pts
-			(xy 229.87 138.43) (xy 226.06 138.43)
+			(xy 62.23 132.08) (xy 69.85 132.08)
 		)
 		(stroke
@@
 	(wire
 		(pts
-			(xy 201.93 86.36) (xy 208.28 86.36)
+			(xy 229.87 138.43) (xy 226.06 138.43)
 		)
 		(stroke
@@
 	(wire
 		(pts
-			(xy 26.67 62.23) (xy 31.75 62.23)
+			(xy 201.93 86.36) (xy 208.28 86.36)
 		)
 		(stroke
@@
 	(wire
 		(pts
-			(xy 44.45 100.33) (xy 44.45 104.14)
+			(xy 26.67 62.23) (xy 31.75 62.23)
 		)
 		(stroke
@@
 	(wire
 		(pts
-			(xy 226.06 127) (xy 229.87 127)
+			(xy 44.45 100.33) (xy 44.45 104.14)
 		)
 		(stroke
@@
 	(wire
 		(pts
-			(xy 173.99 83.82) (xy 163.83 83.82)
+			(xy 226.06 127) (xy 229.87 127)
 		)
 		(stroke
@@
 	(wire
 		(pts
+			(xy 153.67 83.82) (xy 153.67 96.52)
+		)
+		(stroke
+			(width 0)
+			(type default)
+		)
+	)
+	(wire
+		(pts
 			(xy 113.03 29.21) (xy 113.03 20.32)
 		)
@@
 	(wire
 		(pts
+			(xy 153.67 83.82) (xy 173.99 83.82)
+		)
+		(stroke
+			(width 0)
+			(type default)
+		)
+	)
+	(wire
+		(pts
 			(xy 74.93 170.18) (xy 86.36 170.18)
 		)
@@
 	(wire
 		(pts
-			(xy 125.73 29.21) (xy 139.7 29.21)
+			(xy 173.99 88.9) (xy 171.45 88.9)
 		)
 		(stroke
@@
 	(wire
 		(pts
-			(xy 168.91 88.9) (xy 173.99 88.9)
+			(xy 125.73 29.21) (xy 139.7 29.21)
 		)
 		(stroke
@@
 	(wire
 		(pts
-			(xy 88.9 90.17) (xy 88.9 97.79)
-		)
-		(stroke
-			(width 0)
-			(type default)
-		)
-	)
-	(wire
-		(pts
 			(xy 58.42 31.75) (xy 55.88 31.75)
 		)
@@
 	(wire
 		(pts
-			(xy 88.9 97.79) (xy 168.91 97.79)
-		)
-		(stroke
-			(width 0)
-			(type default)
-		)
-	)
-	(wire
-		(pts
 			(xy 171.45 86.36) (xy 171.45 72.39)
 		)
@@
 		)
 	)
+	(wire
+		(pts
+			(xy 171.45 88.9) (xy 171.45 95.25)
+		)
+		(stroke
+			(width 0)
+			(type default)
+		)
+	)
 	(polyline
 		(pts
@@
 	(wire
 		(pts
-			(xy 168.91 97.79) (xy 168.91 88.9)
-		)
-		(stroke
-			(width 0)
-			(type default)
-		)
-	)
-	(wire
-		(pts
 			(xy 153.67 114.3) (xy 153.67 116.84)
 		)
@@
 	(text "Accent"
 		(exclude_from_sim no)
-		(at 187.96 96.52 0)
+		(at 188.468 92.964 0)
 		(effects
 			(font
@@
 	(symbol
 		(lib_id "power:GNDA")
-		(at 163.83 85.09 0)
+		(at 171.45 95.25 0)
 		(unit 1)
 		(exclude_from_sim no)
@@
 		(on_board yes)
 		(dnp no)
+		(fields_autoplaced yes)
 		(property "Reference" "#PWR018"
-			(at 163.83 91.44 0)
+			(at 171.45 101.6 0)
 			(effects
 				(font
@@
 		)
 		(property "Value" "GNDA"
-			(at 159.004 86.36 0)
+			(at 171.45 100.33 0)
 			(effects
 				(font
@@
 		)
 		(property "Footprint" ""
-			(at 163.83 85.09 0)
+			(at 171.45 95.25 0)
 			(effects
 				(font
@@
 		)
 		(property "Datasheet" ""
-			(at 163.83 85.09 0)
+			(at 171.45 95.25 0)
 			(effects
 				(font
@@
 		)
 		(property "Description" "Power symbol creates a global label with name \"GNDA\" , analog ground"
-			(at 163.83 85.09 0)
+			(at 171.45 95.25 0)
 			(effects
 				(font
