File: TBSEQ_Board_V1/analog_separate/組み立てデバッグ前/VCO.kicad_sch (KiCad schematic)
At the start: 30 parts, among them IC11_1 AN6562, J13 Conn_01x01_Pin, Q24 NPN, Q25 NPN, Q26 HN1C01FU-GR,LF_6P DIP, Q27 PNP, Q28 NJFET, Q8 PNP, SW1 2MS1T1B4VS2QES

Commit message: analog_separate fix
実装してバグを修正
・VR6以外のボリュームの左右が逆なのを修正
・デュアルトランジスタをHN1C01FU-GRに変更
・VCA CA3080後の出力段のバイアス/増幅率等の設計ミスを修正
・入力信号のシルク位置が間違っているので修正
⇒それ以外は正常動作を確認済
Parts:
- removed Q26: HN1C01FU-GR,LF_6P DIP, Package_DIP:DIP-6_W7.62mm, symbol SamacSys_Parts:HN1C01FU-GR,LF_6P DIP変換基板_1
- added Q26: HN4C06J-BL_6P DIP, Package_DIP:DIP-6_W7.62mm, symbol SamacSys_Parts:HN4C06J-BL_6P DIP変換基板
Connections:
- net A+5.333V: now also VR2.1 (CCW), Q26.1 (B1); no longer VR2.3 (CW)
- net GNDA: now also VR2.3 (CW); no longer VR2.1 (CCW)
- net at C34.1, IC11_1.2 (-), R102.1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: now also Q26.6 (C1)
- net at R100.1, R100_1.1, R106.1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: now also Q26.3 (B2)
- net at C33.2, Q25.1 (E), Q28.2 (G): now also Q26.4 (C2)
- net at R104.1: now also Q26.2 (E)
Other:
- note added: "HN4C06J-BL_6P DIP"
- note removed: "最終的にはこれに統一 HN1C01FU_DIP"
- moved on the sheet: R104
