File: TBSEQ_Board_V2/mainBorad/MIDIRx.kicad_sch (KiCad schematic)
At the start: 6 parts

Commit message: mainboard
PWS,Digi
Parts:
- DgC1: footprint Capacitor_THT:C_Rect_L7.0mm_W2.0mm_P5.00mm -> Capacitor_SMD:C_0805_2012Metric_Pad1.18x1.45mm_HandSolder
