File: TBSEQ_Board_V2/mainBorad/VCO.kicad_sch (KiCad schematic)
At the start: 28 parts, among them IC11_1 AN6562, J13 Conn_01x01_Pin, Q24 NPN, Q25 NPN, Q26 HN1C01FU-GR,LF_6P DIP, Q27 PNP, Q28 NJFET, Q8 PNP

Commit message: mainboard
部品を全部配置しただけ
Parts:
- J13: footprint Connector_PinHeader_2.54mm:PinHeader_1x01_P2.54mm_Vertical -> Connector_PinHeader_2.54mm:PinHeader_1x01_P2.54mm_Horizontal
Changed lines of the file:
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@@
 			)
 		)
-		(property "Footprint" "Connector_PinHeader_2.54mm:PinHeader_1x01_P2.54mm_Vertical"
+		(property "Footprint" "Connector_PinHeader_2.54mm:PinHeader_1x01_P2.54mm_Horizontal"
 			(at 152.4 45.72 0)
 			(effects
