File: TBSEQ_Board_V2/mainBorad/mainBorad.kicad_pcb (KiCad board)
At the start: 2 copper layers, 109 parts, among them IC11 AN6562, IC12 4066, J7 Conn_01x03_Pin, J8 Conn_01x02_Pin, J9 Conn_01x01_Pin, Q29 NPN, Q30 NPN, Q35 NPN, Q36 PNP, Q37 NPN, Q38 PNP, Q39 NJFET, Q40 NPN, Q41 NPN

Commit message: mainboard
PWS,Digi
Parts:
- removed DgJ6, DgJ7: Conn_01x06, Connector_PinHeader_2.54mm:PinHeader_1x06_P2.54mm_Vertical
- removed VR6: 1M(A), SamacSys_Parts:PTV1113420AA103
- removed VR7: 50K(B), SamacSys_Parts:PTV1113420AA103
- added DgC3: 0.1uF, Capacitor_SMD:C_0805_2012Metric_Pad1.18x1.45mm_HandSolder, B.Cu at (139.3, 71.0)
- added DgC4: 0.1uF, Capacitor_SMD:C_0805_2012Metric_Pad1.18x1.45mm_HandSolder, B.Cu at (148.3, 51.7)
- added DgS2: B3F-1000S, SamacSys_Parts:B3F1060, F.Cu at (121.2, 48.6)
- added VR_J_6: Conn_01x03_Pin, Connector_PinHeader_2.54mm:PinHeader_1x03_P2.54mm_Vertical, F.Cu at (125.2, 102.5)
- added VR_J_7: Conn_01x03_Pin, Connector_PinHeader_2.54mm:PinHeader_1x03_P2.54mm_Vertical, F.Cu at (141.2, 102.5)
- DgC1: footprint Capacitor_THT:C_Rect_L7.0mm_W2.0mm_P5.00mm -> Capacitor_SMD:C_0805_2012Metric_Pad1.18x1.45mm_HandSolder
- DgIC1, DgIC2, DgIC3, DgR1, DgR2: moved to B.Cu
- DgS1: value SKHHLPA010 -> B3F-1000S; footprint SamacSys_Parts:SKHHLPA010 -> SamacSys_Parts:B3F1060
- moved PwF1 120.9 mm to (207.5, 51.9), turned to 180 degrees
- moved PwD1 113.5 mm to (196.6, 57.2), turned to -90 degrees
- moved PwJ2 108.9 mm to (208.1, 41.0), turned to -90 degrees
- moved PwD2 107.3 mm to (202.1, 88.7), turned to -90 degrees
- moved PwC7 101.5 mm to (197.2, 89.2), turned to 180 degrees
- moved PwC9 100.6 mm to (193.5, 76.3), turned to 180 degrees
- moved PwVR1 99.6 mm to (183.7, 102.9), turned to -90 degrees
- moved PwR2 99.1 mm to (194.0, 101.0)
- moved PwJ4 98.8 mm to (208.1, 45.0), turned to -90 degrees
- moved PwD3 95.9 mm to (189.5, 97.5), turned to 90 degrees
- moved PwJ3 94.5 mm to (197.4, 41.2), turned to -90 degrees
- moved DgIC1 94.2 mm to (119.0, 72.1), turned to -90 degrees
- moved PwC4 93.8 mm to (193.4, 71.8), turned to 180 degrees
- moved PwF2 93.7 mm to (179.6, 51.2), turned to 180 degrees
- moved PwC8 93.3 mm to (194.0, 106.9)
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- renumbered C3 to PwC9
Connections:
- DgIC3 pad 11: Net-(DgIC3-Y7) -> unconnected-(DgIC3-Y7-Pad11)
- DgIC3 pad 12: Net-(DgIC3-Y6) -> unconnected-(DgIC3-Y6-Pad12)
- DgIC3 pad 13: Net-(DgIC3-Y5) -> unconnected-(DgIC3-Y5-Pad13)
- DgIC3 pad 14: Net-(DgIC3-Y4) -> unconnected-(DgIC3-Y4-Pad14)
- DgIC3 pad 15: Net-(DgIC3-Y3) -> unconnected-(DgIC3-Y3-Pad15)
- DgIC3 pad 16: Net-(DgIC3-Y2) -> unconnected-(DgIC3-Y2-Pad16)
- DgIC3 pad 4: Net-(DgIC3-A2) -> unconnected-(DgIC3-A2-Pad4)
- DgIC3 pad 5: Net-(DgIC3-A3) -> unconnected-(DgIC3-A3-Pad5)
- DgIC3 pad 6: Net-(DgIC3-A4) -> unconnected-(DgIC3-A4-Pad6)
- DgIC3 pad 7: Net-(DgIC3-A5) -> unconnected-(DgIC3-A5-Pad7)
- DgIC3 pad 8: Net-(DgIC3-A6) -> unconnected-(DgIC3-A6-Pad8)
- DgIC3 pad 9: Net-(DgIC3-A7) -> unconnected-(DgIC3-A7-Pad9)
- DgJ10 pad R1: A+LineOut -> unconnected-(DgJ10-PadR1)
- DgJ10 pad SS1: GNDA -> unconnected-(DgJ10-PadSS1)
- DgJ11 pad 4: A+CV_MIX -> unconnected-(DgJ11-3-Pad4)
- DgJ12 pad 4: A+GATE -> unconnected-(DgJ12-3-Pad4)
- DgJ13 pad 4: A+SyncOut -> unconnected-(DgJ13-3-Pad4)
- DgJ5 pad 5: Net-(DgJ5-Pin_5) -> unconnected-(DgJ5-Pin_5-Pad5)
- DgJ9 pad 2: unconnected-(DgJ9-2_1-Pad2) -> D+5V_SyncIn
- DgJ9 pad 3: D+PlugIn_SyncIn -> D+5V_SyncIn
- DgJ9 pad 4: D+5V_SyncIn -> D+PlugIn_SyncIn
- DgS1 pad 1: Net-(DgU1-RUN) -> Net-(DgS1-COM_1)
- DgS1 pad 2: GNDD -> Net-(DgS1-COM_1)
- DgU1 pad 29: Net-(DgJ5-Pin_5) -> GNDD
- DgU1 pad 30: Net-(DgU1-RUN) -> GNDD
Routing:
- net A+12V: track 0.00 -> 46.4 mm
- net Net-(PwD1-K): track 0.00 -> 36.5 mm
- net A+5.333V: track 0.00 -> 28.0 mm
- net Net-(PwD3-A): track 0.00 -> 25.6 mm
- net Net-(PwJ5-Pin_1): track 0.00 -> 24.2 mm
- net Net-(PwIC1-VIN): track 0.00 -> 12.0 mm
- net Net-(PwIC1-VOUT): track 0.00 -> 7.88 mm
- net Net-(PwJ4-Pin_1): track 0.00 -> 7.14 mm
- net Net-(PwVR1-CCW): track 0.00 -> 6.10 mm
- net D+5V: track 0.00 -> 5.45 mm
Other:
- board outline added: 150 x 250 mm
- board text added: "CCW"
- board text added: "CW"
- board text added: "WIPER"

Commit message: mainBoard
AnInterface
Parts:
- removed DgJ1: Conn_01x04, Connector_PinHeader_2.54mm:PinHeader_1x04_P2.54mm_Vertical
- removed DgJ10: MJ-462, SamacSys_Parts:MJ462
- removed DgJ14, DgJ15: Conn_01x03, Connector_PinHeader_2.54mm:PinHeader_1x03_P2.54mm_Vertical
- removed VR_J_6, VR_J_7: Conn_01x03_Pin, Connector_PinHeader_2.54mm:PinHeader_1x03_P2.54mm_Vertical
- added AnPw1: AnPw, Connector_PinSocket_2.54mm:PinSocket_1x03_P2.54mm_Vertical, F.Cu at (194.7, 113.0)
- added DgPw1: DgPw, Connector_PinSocket_2.54mm:PinSocket_1x03_P2.54mm_Vertical, F.Cu at (89.1, 65.3)
- added PanelJ1: Conn_02x20_Odd_Even, Connector_PinSocket_2.54mm:PinSocket_2x20_P2.54mm_Vertical, F.Cu at (101.1, 82.5)
- DgC4, DgIC3: moved to F.Cu
- moved Q40 80.6 mm to (75.3, 108.5)
- moved C62 80.1 mm to (89.2, 106.0), turned to -90 degrees
- moved Q41 76.3 mm to (81.5, 108.4)
- moved DgIC3 75.6 mm to (78.0, 56.0), turned to 0 degrees
- moved Q39 75.0 mm to (78.9, 114.5)
- moved R107 73.0 mm to (185.2, 113.3), turned to 90 degrees
- moved DgC4 70.1 mm to (78.2, 51.3), turned to 180 degrees
- moved C55 69.8 mm to (93.4, 99.8), turned to -90 degrees
- moved R91 69.4 mm to (179.3, 95.8)
- moved R93 69.1 mm to (179.5, 104.9)
- moved DgJ8 67.6 mm to (77.7, 35.2)
- moved DgC1 66.9 mm to (96.0, 44.1)
- moved DgIC4 66.9 mm to (86.5, 44.4)
- moved DgR4 66.9 mm to (92.5, 44.0)
- moved DgD1 66.9 mm to (79.7, 44.7)
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Connections:
- net Net-(D28-A) renamed A_VR6_WIPER_CW
- net Net-(VR_J_6-Pin_1) renamed A_VR6_CCW
- DgJ16 pad 2: A+SLIDE -> A+CV_MIX
- DgJ16 pad 3: A-ACC -> A+SLIDE
- DgJ16 pad 4: A+GATE -> A-ACC
- DgJ16 pad 5: A+CV_MIX -> A+GATE
- DgS1 pad 1: Net-(DgS1-COM_1) -> GNDD
- DgS1 pad 2: Net-(DgS1-COM_1) -> GNDD
- DgS1 pad 3: GNDD -> Net-(DgS1-N.O._1)
- DgS1 pad 4: GNDD -> Net-(DgS1-N.O._1)
- DgS2 pad 1: Net-(DgS2-COM_1) -> GNDD
- DgS2 pad 2: Net-(DgS2-COM_1) -> GNDD
- DgS2 pad 3: GNDD -> Net-(DgS2-N.O._1)
- DgS2 pad 4: GNDD -> Net-(DgS2-N.O._1)
- DgU1 pad 29: GNDD -> Net-(DgS2-N.O._1)
- DgU1 pad 30: GNDD -> Net-(DgS1-N.O._1)
- IC12 pad 8: Net-(VR_J_7-Pin_3) -> A_VR7_CW
- R141 pad 1: D-ACC -> A-ACC
- R146 pad 1: D+GATE -> A+GATE
- R59 pad 1: D+SLIDE -> A+SLIDE
Routing:
- net Net-(PwJ5-Pin_1): track 24.2 -> 0.14 mm
- net Net-(PwIC1-VIN): track 12.0 -> 0.03 mm
- net A+12V: track 46.4 -> 54.5 mm
- net Net-(PwIC1-VOUT): track 7.88 -> 0.00 mm
- net D+5V: track 5.45 -> 0.00 mm
- net (no net): vias 0 -> 46
- added copper zone on B.Cu, net ADAPTER GND
- added copper zone on F.Cu, net ADAPTER GND
- added copper zone on B.Cu, net GNDA
- added copper zone on F.Cu, net GNDA
- added copper zone on B.Cu, net GNDD
- added copper zone on F.Cu, net GNDD
Other:
- outline, holes or cut-outs redrawn
- board text added: "A+CV"
- board text added: "A+CV_MIX"
- board text added: "A+GATE"
- board text added: "A+SLIDE"
- board text added: "A-ACC"
- board text removed: "CCW"
- board text removed: "CW"
- board text removed: "WIPER"

Commit message: mainBoard
VCO
Parts:
- added C10: 0.01uF, Capacitor_THT:C_Rect_L7.2mm_W2.5mm_P5.00mm_FKS2_FKP2_MKS2_MKP2, F.Cu at (191.1, 150.3)
- added C11: 1uF/50V, Capacitor_THT:CP_Radial_D5.0mm_P2.00mm, F.Cu at (181.6, 156.5)
- added C33: 0.01uF, Capacitor_THT:C_Rect_L7.2mm_W2.5mm_P5.00mm_FKS2_FKP2_MKS2_MKP2, F.Cu at (199.4, 150.3)
- added C34: 0.001uF, Capacitor_THT:C_Rect_L7.2mm_W2.5mm_P5.00mm_FKS2_FKP2_MKS2_MKP2, F.Cu at (203.8, 124.5)
- added D25: D, Diode_THT:D_A-405_P2.54mm_Vertical_AnodeUp, F.Cu at (170.8, 132.7)
- added IC11_1: AN6562, Package_DIP:DIP-8_W7.62mm, F.Cu at (197.5, 130.2)
- added J13: Conn_01x01_Pin, Connector_PinHeader_2.54mm:PinHeader_1x01_P2.54mm_Vertical, F.Cu at (145.4, 115.6)
- added Q24: NPN, Package_TO_SOT_THT:TO-92_HandSolder, F.Cu at (177.2, 126.4)
- added Q25: NPN, Package_TO_SOT_THT:TO-92_HandSolder, F.Cu at (170.8, 126.4)
- added Q26: HN1C01FU-GR,LF_6P DIP, Package_DIP:DIP-6_W7.62mm, F.Cu at (184.2, 130.2)
- added Q27: PNP, Package_TO_SOT_THT:TO-92_HandSolder, F.Cu at (177.2, 134.0)
- added Q28: NJFET, Package_TO_SOT_THT:TO-92_HandSolder, F.Cu at (198.8, 159.8)
- added Q8: PNP, Package_TO_SOT_THT:TO-92_HandSolder, F.Cu at (180.3, 152.2)
- added R100: 1K(TEMPCO), Resistor_THT:R_Axial_DIN0207_L6.3mm_D2.5mm_P2.54mm_Vertical, F.Cu at (189.2, 139.7)
- added R100_1: 1K(TEMPCO), Resistor_THT:R_Axial_DIN0207_L6.3mm_D2.5mm_P2.54mm_Vertical, F.Cu at (189.2, 142.9)
- added R101: 10K, Resistor_THT:R_Axial_DIN0207_L6.3mm_D2.5mm_P2.54mm_Vertical, F.Cu at (179.3, 138.4)
- added R102: 100K, Resistor_THT:R_Axial_DIN0207_L6.3mm_D2.5mm_P2.54mm_Vertical, F.Cu at (197.7, 120.0)
- added R103: 220K, Resistor_THT:R_Axial_DIN0207_L6.3mm_D2.5mm_P2.54mm_Vertical, F.Cu at (205.3, 120.0)
- added R104: 2.2K, Resistor_THT:R_Axial_DIN0207_L6.3mm_D2.5mm_P2.54mm_Vertical, F.Cu at (198.1, 142.9)
- added R105: 10K, Resistor_THT:R_Axial_DIN0207_L6.3mm_D2.5mm_P2.54mm_Vertical, F.Cu at (195.6, 153.2)
- added R106: 27K, Resistor_THT:R_Axial_DIN0207_L6.3mm_D2.5mm_P2.54mm_Vertical, F.Cu at (184.8, 123.8)
- added R118: 100K, Resistor_THT:R_Axial_DIN0207_L6.3mm_D2.5mm_P2.54mm_Vertical, F.Cu at (192.4, 123.8)
- added R34: 10K, Resistor_THT:R_Axial_DIN0207_L6.3mm_D2.5mm_P2.54mm_Vertical, F.Cu at (186.7, 152.8)
- added R35: 100K, Resistor_THT:R_Axial_DIN0207_L6.3mm_D2.5mm_P2.54mm_Vertical, F.Cu at (186.7, 156.2)
- added R36: 10K, Resistor_THT:R_Axial_DIN0207_L6.3mm_D2.5mm_P2.54mm_Vertical, F.Cu at (176.5, 152.8)
- added R45: 22K, Resistor_THT:R_Axial_DIN0207_L6.3mm_D2.5mm_P2.54mm_Vertical, F.Cu at (176.5, 158.3)
- added TM4: 50K, SamacSys_Parts:3006P1503LF, F.Cu at (196.8, 109.9)
- added TM5: 5K, SamacSys_Parts:3006P1503LF, F.Cu at (196.6, 100.7)
- moved AnPw1 42.0 mm to (184.2, 72.4), turned to 180 degrees
- moved PwC8 23.3 mm to (199.4, 86.4), turned to -90 degrees
- moved PwVR1 20.8 mm to (188.7, 85.1), turned to 0 degrees
- moved PwC7 19.0 mm to (201.3, 73.7)
- moved PwC6 18.7 mm to (192.3, 73.7)
- moved PwIC3 18.3 mm to (207.4, 80.3)
- moved PwR1 17.6 mm to (195.9, 81.6)
- moved PwD3 17.6 mm to (201.2, 82.0)
- moved PwR2 17.5 mm to (206.8, 85.7), turned to 180 degrees
- moved PwC2 10.9 mm to (194.1, 54.0), turned to 180 degrees
- moved PwIC2 9.01 mm to (197.1, 62.2)
- moved PwC9 9.01 mm to (194.1, 67.3)
- moved PwC4 9.01 mm to (194.0, 62.8)
- moved C55 7.44 mm to (86.0, 99.8)
- moved R148 7.44 mm to (97.2, 93.3)
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Connections:
- net Net-(PwD1-K) renamed A+15V
- net Net-(PwIC1-VIN) renamed D+15V
- net Net-(PwJ4-Pin_1) renamed A+15VPre
- net Net-(PwJ5-Pin_1) renamed D+15VPre
- PanelJ1 pad 17: A_VR2_CCW -> GNDA
- PanelJ1 pad 21: A_VR2_CW -> A+5.333V
- PanelJ1 pad 29: GNDA -> A+VCO_SQU
- PanelJ1 pad 31: GNDA -> A+VCO_SAW
- PanelJ1 pad 33: GNDA -> A+VCO_WAVE
Routing:
- net A+12V: track 54.5 -> 0.00 mm
- net A+15V: track 36.5 -> 0.00 mm
- net A+5.333V: track 28.0 -> 0.00 mm
- net Net-(PwD3-A): track 25.6 -> 0.00 mm
- net Net-(PwVR1-CCW): track 6.10 -> 0.00 mm
Other:
- outline, holes or cut-outs redrawn
- board text added: "TUNE"
- board text added: "WIDTH"

Commit message: mainboard
部品を全部配置しただけ
Parts:
- added C13: 1uF/50V, Capacitor_THT:CP_Radial_D5.0mm_P2.00mm, F.Cu at (141.3, 98.5)
- added C14: 1uF/50V, Capacitor_THT:CP_Radial_D5.0mm_P2.00mm, F.Cu at (113.6, 162.3)
- added C15: 1uF/50V, Capacitor_THT:CP_Radial_D5.0mm_P2.00mm, F.Cu at (131.5, 140.1)
- added C16: 10uF/16V, Capacitor_THT:CP_Radial_D4.0mm_P2.00mm, F.Cu at (161.0, 128.8)
- added C17: 1uF/50V, Capacitor_THT:CP_Radial_D5.0mm_P2.00mm, F.Cu at (173.4, 123.5)
- added C18: 0.018uF, Capacitor_THT:C_Rect_L7.2mm_W2.5mm_P5.00mm_FKS2_FKP2_MKS2_MKP2, F.Cu at (171.4, 141.4)
- added C19: 0.033uF, Capacitor_THT:C_Rect_L7.2mm_W2.5mm_P5.00mm_FKS2_FKP2_MKS2_MKP2, F.Cu at (171.4, 154.4)
- added C20: 0.01uF, Capacitor_THT:C_Rect_L7.2mm_W2.5mm_P5.00mm_FKS2_FKP2_MKS2_MKP2, F.Cu at (102.3, 151.9)
- added C21: 0.01uF, Capacitor_THT:C_Rect_L7.2mm_W2.5mm_P5.00mm_FKS2_FKP2_MKS2_MKP2, F.Cu at (102.3, 148.6)
- added C22: 1uF/50V, Capacitor_THT:CP_Radial_D5.0mm_P2.00mm, F.Cu at (124.5, 134.5)
- added C23: 1uF/50V, Capacitor_THT:CP_Radial_D5.0mm_P2.00mm, F.Cu at (151.2, 148.9)
- added C24: 0.033uF, Capacitor_THT:C_Rect_L7.2mm_W2.5mm_P5.00mm_FKS2_FKP2_MKS2_MKP2, F.Cu at (171.4, 162.5)
- added C25: 0.1uF, Capacitor_THT:C_Rect_L7.2mm_W2.5mm_P5.00mm_FKS2_FKP2_MKS2_MKP2, F.Cu at (142.1, 149.8)
- added C26: 0.033uF, Capacitor_THT:C_Rect_L7.2mm_W2.5mm_P5.00mm_FKS2_FKP2_MKS2_MKP2, F.Cu at (169.0, 165.7)
- added C27: 0.1uF, Capacitor_THT:C_Rect_L7.2mm_W2.5mm_P5.00mm_FKS2_FKP2_MKS2_MKP2, F.Cu at (142.1, 146.4)
- added C28: 47uF/16V, Capacitor_THT:CP_Radial_D4.0mm_P2.00mm, F.Cu at (136.6, 159.6)
- added C29: 1uF/50V, Capacitor_THT:CP_Radial_D5.0mm_P2.00mm, F.Cu at (119.7, 162.4)
- added C30: 10uF/16V, Capacitor_THT:CP_Radial_D4.0mm_P2.00mm, F.Cu at (136.7, 164.7)
- added C36: 0.033uF, Capacitor_THT:C_Rect_L7.2mm_W2.5mm_P5.00mm_FKS2_FKP2_MKS2_MKP2, F.Cu at (96.3, 121.8)
- added C37: 10uF/16V, Capacitor_THT:CP_Radial_D4.0mm_P2.00mm, F.Cu at (97.4, 161.0)
- added C41: 0.1uF, Capacitor_THT:C_Rect_L7.2mm_W2.5mm_P5.00mm_FKS2_FKP2_MKS2_MKP2, F.Cu at (115.1, 143.0)
- added C42: 1uF/50V, Capacitor_THT:CP_Radial_D5.0mm_P2.00mm, F.Cu at (107.7, 127.6)
- added D24: D, Diode_THT:D_A-405_P2.54mm_Vertical_AnodeUp, F.Cu at (141.3, 136.1)
- added D27: D, Diode_THT:D_A-405_P2.54mm_Vertical_AnodeUp, F.Cu at (95.1, 133.2)
- added D35: D, Diode_THT:D_A-405_P2.54mm_Vertical_AnodeUp, F.Cu at (102.2, 125.9)
- added D36: D, Diode_THT:D_A-405_P2.54mm_Vertical_AnodeUp, F.Cu at (117.1, 125.6)
- added IC15: CA3080A, Package_DIP:DIP-8_W7.62mm, F.Cu at (87.5, 161.2)
- added J3: Conn_01x02_Pin, Connector_PinHeader_2.54mm:PinHeader_1x02_P2.54mm_Horizontal, F.Cu at (106.3, 158.8)
- added J4: Conn_01x02_Pin, Connector_PinHeader_2.54mm:PinHeader_1x02_P2.54mm_Horizontal, F.Cu at (79.2, 120.1)
- added Q10: PNP, Package_TO_SOT_THT:TO-92_HandSolder, F.Cu at (151.5, 141.2)
- added Q11: NPN, Package_TO_SOT_THT:TO-92_HandSolder, F.Cu at (151.5, 136.0)
- added Q12: HN1C01FU-GR,LF_6P DIP, Package_DIP:DIP-6_W7.62mm, F.Cu at (178.1, 130.3)
- added Q13: NPN, Package_TO_SOT_THT:TO-92_HandSolder, F.Cu at (166.3, 142.6)
- added Q14: NPN, Package_TO_SOT_THT:TO-92_HandSolder, F.Cu at (166.4, 150.2)
- added Q15: NPN, Package_TO_SOT_THT:TO-92_HandSolder, F.Cu at (176.8, 142.6)
- added Q16: NPN, Package_TO_SOT_THT:TO-92_HandSolder, F.Cu at (166.3, 158.8)
- added Q17: NPN, Package_TO_SOT_THT:TO-92_HandSolder, F.Cu at (176.7, 150.2)
- added Q18: NPN, Package_TO_SOT_THT:TO-92_HandSolder, F.Cu at (133.3, 131.8)
- added Q19: NPN, Package_TO_SOT_THT:TO-92_HandSolder, F.Cu at (108.9, 155.0)
- added Q20: NPN, Package_TO_SOT_THT:TO-92_HandSolder, F.Cu at (114.6, 148.8)
- added Q21: HN1C01FU-GR,LF_6P DIP, Package_DIP:DIP-6_W7.62mm, F.Cu at (124.4, 146.5)
- added Q22: HN1C01FU-GR,LF_6P DIP, Package_DIP:DIP-6_W7.62mm, F.Cu at (145.0, 155.9)
- added Q23: NPN, Package_TO_SOT_THT:TO-92_HandSolder, F.Cu at (176.6, 158.8)
- added Q31: PNP, Package_TO_SOT_THT:TO-92_HandSolder, F.Cu at (100.0, 138.2)
- added Q32: NPN, Package_TO_SOT_THT:TO-92_HandSolder, F.Cu at (115.0, 134.3)
- added Q9: PNP, Package_TO_SOT_THT:TO-92_HandSolder, F.Cu at (151.5, 130.7)
- added R108: 2.2K, Resistor_THT:R_Axial_DIN0207_L6.3mm_D2.5mm_P2.54mm_Vertical, F.Cu at (114.7, 154.8)
- added R109: 10K, Resistor_THT:R_Axial_DIN0207_L6.3mm_D2.5mm_P2.54mm_Vertical, F.Cu at (119.8, 154.7)
- added R110: 22K, Resistor_THT:R_Axial_DIN0207_L6.3mm_D2.5mm_P2.54mm_Vertical, F.Cu at (129.8, 158.1)
- added R111: 22K, Resistor_THT:R_Axial_DIN0207_L6.3mm_D2.5mm_P2.54mm_Vertical, F.Cu at (129.8, 163.5)
- added R112: 10K, Resistor_THT:R_Axial_DIN0207_L6.3mm_D2.5mm_P2.54mm_Vertical, F.Cu at (119.8, 143.7)
- added R113: 100K, Resistor_THT:R_Axial_DIN0207_L6.3mm_D2.5mm_P2.54mm_Vertical, F.Cu at (119.8, 149.0)
- added R114: 100K, Resistor_THT:R_Axial_DIN0207_L6.3mm_D2.5mm_P2.54mm_Vertical, F.Cu at (124.8, 158.0)
- added R115: 10K, Resistor_THT:R_Axial_DIN0207_L6.3mm_D2.5mm_P2.54mm_Vertical, F.Cu at (141.1, 160.9)
- added R116: 10K, Resistor_THT:R_Axial_DIN0207_L6.3mm_D2.5mm_P2.54mm_Vertical, F.Cu at (124.8, 163.5)
- added R119: 47K, Resistor_THT:R_Axial_DIN0207_L6.3mm_D2.5mm_P2.54mm_Vertical, F.Cu at (92.9, 125.9)
- added R120: 22K, Resistor_THT:R_Axial_DIN0207_L6.3mm_D2.5mm_P2.54mm_Vertical, F.Cu at (94.9, 129.7)
- added R121: 220K, Resistor_THT:R_Axial_DIN0207_L6.3mm_D2.5mm_P2.54mm_Vertical, F.Cu at (92.1, 148.5)
- added R122: 100K, Resistor_THT:R_Axial_DIN0207_L6.3mm_D2.5mm_P2.54mm_Vertical, F.Cu at (92.1, 151.9)
- added R123: 1.5M, Resistor_THT:R_Axial_DIN0207_L6.3mm_D2.5mm_P2.54mm_Vertical, F.Cu at (109.6, 137.2)
- added R124: 2.2K, Resistor_THT:R_Axial_DIN0207_L6.3mm_D2.5mm_P2.54mm_Vertical, F.Cu at (90.7, 161.2)
- added R125: 2.2K, Resistor_THT:R_Axial_DIN0207_L6.3mm_D2.5mm_P2.54mm_Vertical, F.Cu at (90.6, 157.6)
- added R126: 2.2K, Resistor_THT:R_Axial_DIN0207_L6.3mm_D2.5mm_P2.54mm_Vertical, F.Cu at (96.2, 157.6)
- added R130: 100, Resistor_THT:R_Axial_DIN0207_L6.3mm_D2.5mm_P2.54mm_Vertical, F.Cu at (119.7, 138.4)
- added R131: 220K, Resistor_THT:R_Axial_DIN0207_L6.3mm_D2.5mm_P2.54mm_Vertical, F.Cu at (102.1, 133.1)
- added R132: 100, Resistor_THT:R_Axial_DIN0207_L6.3mm_D2.5mm_P2.54mm_Vertical, F.Cu at (107.6, 133.0)
- added R133: 2.2K, Resistor_THT:R_Axial_DIN0207_L6.3mm_D2.5mm_P2.54mm_Vertical, F.Cu at (100.0, 129.5)
- added R134: 22K, Resistor_THT:R_Axial_DIN0207_L6.3mm_D2.5mm_P2.54mm_Vertical, F.Cu at (117.1, 129.1)
- added R46: 47K, Resistor_THT:R_Axial_DIN0207_L6.3mm_D2.5mm_P2.54mm_Vertical, F.Cu at (139.2, 132.6)
- added R47: 10K, Resistor_THT:R_Axial_DIN0207_L6.3mm_D2.5mm_P2.54mm_Vertical, F.Cu at (139.3, 125.8)
- added R61: 10K, Resistor_THT:R_Axial_DIN0207_L6.3mm_D2.5mm_P2.54mm_Vertical, F.Cu at (139.2, 129.2)
- added R62: 220K, Resistor_THT:R_Axial_DIN0207_L6.3mm_D2.5mm_P2.54mm_Vertical, F.Cu at (178.3, 123.4)
- added R63: 220K, Resistor_THT:R_Axial_DIN0207_L6.3mm_D2.5mm_P2.54mm_Vertical, F.Cu at (146.0, 132.5)
- added R64: 10K, Resistor_THT:R_Axial_DIN0207_L6.3mm_D2.5mm_P2.54mm_Vertical, F.Cu at (148.1, 125.8)
- added R65: 10K, Resistor_THT:R_Axial_DIN0207_L6.3mm_D2.5mm_P2.54mm_Vertical, F.Cu at (151.9, 125.8)
- added R66: 100K, Resistor_THT:R_Axial_DIN0207_L6.3mm_D2.5mm_P2.54mm_Vertical, F.Cu at (124.8, 125.6)
- added R67: 2.2K, Resistor_THT:R_Axial_DIN0207_L6.3mm_D2.5mm_P2.54mm_Vertical, F.Cu at (133.8, 135.3)
- added R68: 2.2K, Resistor_THT:R_Axial_DIN0207_L6.3mm_D2.5mm_P2.54mm_Vertical, F.Cu at (165.2, 129.1)
- added R69: 2.2K, Resistor_THT:R_Axial_DIN0207_L6.3mm_D2.5mm_P2.54mm_Vertical, F.Cu at (161.2, 134.5)
- added R70: 2.2K, Resistor_THT:R_Axial_DIN0207_L6.3mm_D2.5mm_P2.54mm_Vertical, F.Cu at (168.5, 131.2)
- added R71: 2.2K, Resistor_THT:R_Axial_DIN0207_L6.3mm_D2.5mm_P2.54mm_Vertical, F.Cu at (148.1, 129.2)
- added R72: 100K, Resistor_THT:R_Axial_DIN0207_L6.3mm_D2.5mm_P2.54mm_Vertical, F.Cu at (146.0, 135.9)
- added R73: 100K, Resistor_THT:R_Axial_DIN0207_L6.3mm_D2.5mm_P2.54mm_Vertical, F.Cu at (148.0, 139.6)
- added R94: 10K, Resistor_THT:R_Axial_DIN0207_L6.3mm_D2.5mm_P2.54mm_Vertical, F.Cu at (133.9, 125.6)
- added R95: 100, Resistor_THT:R_Axial_DIN0207_L6.3mm_D2.5mm_P2.54mm_Vertical, F.Cu at (138.8, 154.0)
- added R96: 10K, Resistor_THT:R_Axial_DIN0207_L6.3mm_D2.5mm_P2.54mm_Vertical, F.Cu at (107.4, 149.0)
- added R97: 10K, Resistor_THT:R_Axial_DIN0207_L6.3mm_D2.5mm_P2.54mm_Vertical, F.Cu at (161.9, 144.6)
- added R98: 2.2K, Resistor_THT:R_Axial_DIN0207_L6.3mm_D2.5mm_P2.54mm_Vertical, F.Cu at (165.1, 136.5)
- added R99: 100K, Resistor_THT:R_Axial_DIN0207_L6.3mm_D2.5mm_P2.54mm_Vertical, F.Cu at (126.9, 129.3)
- added TM3: 500K, SamacSys_Parts:3006P1503LF, F.Cu at (159.4, 151.3)
- added VCA_C_1: 10uF/16V, Capacitor_THT:CP_Radial_D4.0mm_P2.00mm, F.Cu at (81.4, 142.4)
- added VCA_C_2: 10uF/16V, Capacitor_THT:CP_Radial_D4.0mm_P2.00mm, F.Cu at (75.2, 156.0)
- added VCA_IC_1: Opamp_Dual, Package_DIP:DIP-8_W7.62mm, F.Cu at (83.4, 137.8)
- added VCA_R1: 10K, Resistor_THT:R_Axial_DIN0207_L6.3mm_D2.5mm_P2.54mm_Vertical, F.Cu at (87.5, 132.5)
- added VCA_R2: 100, Resistor_THT:R_Axial_DIN0207_L6.3mm_D2.5mm_P2.54mm_Vertical, F.Cu at (86.5, 142.4)
- added VCA_R3: 47K, Resistor_THT:R_Axial_DIN0207_L6.3mm_D2.5mm_P2.54mm_Vertical, F.Cu at (86.5, 137.9)
- added VCA_R4: 100K, Resistor_THT:R_Axial_DIN0207_L6.3mm_D2.5mm_P2.54mm_Vertical, F.Cu at (72.7, 138.0)
- added VCA_R5: 47K, Resistor_THT:R_Axial_DIN0207_L6.3mm_D2.5mm_P2.54mm_Vertical, F.Cu at (85.3, 148.2)
- added VCA_R6: 100K, Resistor_THT:R_Axial_DIN0207_L6.3mm_D2.5mm_P2.54mm_Vertical, F.Cu at (73.9, 148.2)
- added VCA_R7: 100K, Resistor_THT:R_Axial_DIN0207_L6.3mm_D2.5mm_P2.54mm_Vertical, F.Cu at (79.5, 148.2)
- J13, J9: footprint Connector_PinHeader_2.54mm:PinHeader_1x01_P2.54mm_Vertical -> Connector_PinHeader_2.54mm:PinHeader_1x01_P2.54mm_Horizontal
- J7: footprint Connector_PinHeader_2.54mm:PinHeader_1x03_P2.54mm_Vertical -> Connector_PinHeader_2.54mm:PinHeader_1x03_P2.54mm_Horizontal
- J8: footprint Connector_PinHeader_2.54mm:PinHeader_1x02_P2.54mm_Vertical -> Connector_PinHeader_2.54mm:PinHeader_1x02_P2.54mm_Horizontal
- moved J8 73.0 mm to (79.0, 109.5), turned to 180 degrees
- moved J13 57.6 mm to (184.3, 158.1), turned to -90 degrees
- moved J7 46.6 mm to (79.1, 98.6), turned to 180 degrees
- moved J9 25.4 mm to (203.6, 95.9)
- moved DgJ16 20.8 mm to (175.1, 57.9), turned to 0 degrees
- moved C11 18.4 mm to (199.9, 158.6)
- moved D25 18.2 mm to (185.5, 143.5), turned to -90 degrees
- moved R45 17.7 mm to (194.1, 160.7), turned to 180 degrees
- moved R100 14.8 mm to (196.8, 127.0)
- moved Q25 14.6 mm to (184.5, 131.4)
- moved R36 14.0 mm to (190.4, 150.6)
- moved R101 13.0 mm to (190.4, 145.2), turned to 90 degrees
- moved R35 12.2 mm to (195.4, 147.6), turned to 0 degrees
- moved R105 12.0 mm to (206.9, 149.0), turned to 0 degrees
- moved Q8 12.0 mm to (191.6, 156.3)
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Connections:
- PanelJ1 pad 11: A_VR8_CCW -> unconnected-(PanelJ1-Pin_11-Pad11)
- PanelJ1 pad 13: A_VR8_WIPER -> A+LineOut
- PanelJ1 pad 15: A_VR8_CW -> unconnected-(PanelJ1-Pin_15-Pad15)
- PanelJ1 pad 22: A_VR3_CW -> A+12V
- PanelJ1 pad 23: A_VR4_1_CCW -> GNDA
- PanelJ1 pad 25: A_VR4_1_WIPER -> A+VCA_Resonance
- PanelJ1 pad 27: A_VR4_1_CW -> A+VCA_Signal
- PanelJ1 pad 34: A_VR5_CW -> A+ENV.MOD
Routing:
- net (no net): vias 46 -> 0
Other:
- board size 150 x 250 mm -> 150 x 150 mm
- board text added: "FREQ"
- board text added: "VCO CV"
- board text added: "VCO WAVE"
