File: TBSEQ_Board_V2/mainBorad/LevelConvert.kicad_sch (KiCad schematic)
At the start: 4 parts

Commit message: mainboard
PWS,Digi
Parts:
- removed DgJ6, DgJ7: Conn_01x06, Connector_PinHeader_2.54mm:PinHeader_1x06_P2.54mm_Vertical, symbol Connector_Generic:Conn_01x06
- added DgC3, DgC4: 0.1uF, Capacitor_SMD:C_0805_2012Metric_Pad1.18x1.45mm_HandSolder, symbol Device:C
- DgIC3: footprint SamacSys_Parts:SOP65P640X110-20N -> SOP65P640X110-20N
Connections:
- net D+3.3V: now also DgC4.1
- net D+5V: now also DgC3.1
- net GNDD: now also DgC3.2, DgC4.2
- no-connect marks 0 -> 12

Commit message: mainBoradV2.5
修正中
Parts:
- removed DgIC2: 74HC126D, SamacSys_Parts:SOIC127P600X175-14N, symbol SamacSys_Parts:74HC126D
- added DgIC2: TC74VHC541FK, SamacSys_Parts:SOP50P400X100-20N, symbol SamacSys_Parts:TC74VHC541FK
- added V05_IN_J, V05_OUT_J: Conn_01x03, Connector_PinSocket_1.27mm:PinSocket_1x03_P1.27mm_Vertical, symbol Connector_Generic:Conn_01x03
- added V33_IN_J, V33_OUT_J1: Conn_01x05, Connector_PinHeader_1.27mm:PinHeader_1x05_P1.27mm_Vertical, symbol Connector_Generic:Conn_01x05
Connections:
- net A+GATE: now also DgIC2.18 (Y1)
- net A+SLIDE: now also DgIC2.17 (Y2)
- net A+SyncOut: now also DgIC2.15 (Y4)
- net A-ACC: now also DgIC2.16 (Y3)
- net D+5V: now also DgIC2.20 (VCC)
- net D+GATE: now also DgIC2.2 (A1)
- net D+SLIDE: now also DgIC2.3 (A2)
- net D+SyncOut: now also DgIC2.5 (A4)
- net D-ACC: now also DgIC2.4 (A3)
- net GNDD: now also DgIC2.1 (~{G1}), DgIC2.10 (GND), DgIC2.19 (~{G2})
- net at DgIC3.11 (Y7): now also V33_OUT_J1.5 (Pin_5)
- net at DgIC3.12 (Y6): now also V33_OUT_J1.4 (Pin_4)
- net at DgIC3.13 (Y5): now also V33_OUT_J1.3 (Pin_3)
- net at DgIC3.14 (Y4): now also V33_OUT_J1.2 (Pin_2)
- net at DgIC3.15 (Y3): now also V33_OUT_J1.1 (Pin_1)
- net D+SyncIn_Run/Stop: now reaches DgIC3.16 (Y2)
- net D+5V_SyncIn_Run/Stop: now reaches DgIC3.4 (A2)
- net at DgIC3.5 (A3): now also V33_IN_J.1 (Pin_1)
- net at DgIC3.6 (A4): now also V33_IN_J.2 (Pin_2)
- net at DgIC3.7 (A5): now also V33_IN_J.3 (Pin_3)
- net at DgIC3.8 (A6): now also V33_IN_J.4 (Pin_4)
- net at DgIC3.9 (A7): now also V33_IN_J.5 (Pin_5)
- new net: DgIC2.13 (Y6), V05_OUT_J.1 (Pin_1)
- new net: DgIC2.12 (Y7), V05_OUT_J.2 (Pin_2)
- new net: DgIC2.11 (Y8), V05_OUT_J.3 (Pin_3)
- new net: DgIC2.7 (A6), V05_IN_J.1 (Pin_1)
- new net: DgIC2.8 (A7), V05_IN_J.2 (Pin_2)
- new net: DgIC2.9 (A8), V05_IN_J.3 (Pin_3)
- new net A+SyncOut_Run/Stop: DgIC2.14 (Y5)
- new net D+SyncOut_Run/Stop: DgIC2.6 (A5)
- no-connect marks 12 -> 0
Other:
- moved on the sheet: DgC3
