File: TBSEQ_Board_V2/mainBorad/RasPico.kicad_sch (KiCad schematic)
At the start: 10 parts

Commit message: mainboard
PWS,Digi
Parts:
- removed DgS1: SKHHLPA010, SamacSys_Parts:SKHHLPA010, symbol SamacSys_Parts:SKHHLPA010
- added DgS1, DgS2: B3F-1000S, SamacSys_Parts:B3F1060, symbol SamacSys_Parts:B3F-1000S
Connections:
- net GNDD: now also DgU1.29 (GP22), DgU1.30 (RUN), DgS1.3 (N.O._1), DgS1.4 (N.O._2), DgS2.3 (N.O._1), DgS2.4 (N.O._2)
- net at DgJ5.5 (Pin_5): no longer DgU1.29 (GP22)
- new net: DgS1.1 (COM_1), DgS1.2 (COM_2)
- new net: DgS2.1 (COM_1), DgS2.2 (COM_2)
- no-connect marks 2 -> 3
Other:
- note added: "Test Button"

Commit message: mainBoard
AnInterface
Parts:
- removed DgJ1: Conn_01x04, Connector_PinHeader_2.54mm:PinHeader_1x04_P2.54mm_Vertical, symbol Connector_Generic:Conn_01x04
Connections:
- net GNDD: now also DgS1.1 (COM_1), DgS1.2 (COM_2), DgS2.1 (COM_1), DgS2.2 (COM_2); no longer DgS1.3 (N.O._1), DgS1.4 (N.O._2), DgS2.3 (N.O._1), DgS2.4 (N.O._2), DgU1.29 (GP22), DgU1.30 (RUN)
- new net: DgS2.3 (N.O._1), DgS2.4 (N.O._2), DgU1.29 (GP22)
- new net: DgS1.3 (N.O._1), DgS1.4 (N.O._2), DgU1.30 (RUN)

Commit message: mainBoradV2.5
修正中
Parts:
- removed DgJ2, DgJ4: Conn_01x04, Connector_PinHeader_2.54mm:PinHeader_1x04_P2.54mm_Vertical, symbol Connector_Generic:Conn_01x04
- removed DgU2: IRLML6402(DIP6Convert), Package_DIP:DIP-6_W7.62mm, symbol SamacSys_Parts:IRLML6402(DIP6_Convert)
- added DgJ2: Conn_01x07, Connector_PinHeader_2.54mm:PinHeader_1x07_P2.54mm_Vertical, symbol Connector_Generic:Conn_01x07
- added DgU2: IRLML6402, Package_TO_SOT_SMD:SOT-23W_Handsoldering, symbol Transistor_FET:IRLML6402
Connections:
- net D+3.3V_MIDIRX: now also DgJ3.2 (Pin_2), DgU1.2 (GP1); no longer DgU1.16 (GP12)
- net D+5V: now also DgU2.3 (D)
- net D+VBUS: now also DgU2.1 (G)
- net D+VSYS: now also DgU2.2 (S)
- net at DgU1.10 (GP7): now also DgJ2.2 (Pin_2)
- net at DgU1.11 (GP8): now also DgJ2.3 (Pin_3)
- net at DgU1.12 (GP9): now also DgJ2.4 (Pin_4)
- net at DgU1.14 (GP10): now also DgJ2.5 (Pin_5)
- net at DgU1.15 (GP11): now also DgJ2.6 (Pin_6)
- net D+SyncIn_Run/Stop: now reaches DgU1.17 (GP13)
- net D+SyncOut_Run/Stop: now reaches DgU1.19 (GP14)
- net at DgU1.9 (GP6): now also DgJ2.1 (Pin_1)
- new net: DgJ2.7 (Pin_7), DgU1.16 (GP12)
