File: TBSEQ_Board_V3/mainBorad/MIDIRx.kicad_sch (KiCad schematic)
At the start: 6 parts

Commit message: V3Board
アートワーク中
Parts:
- added DgJ1: KDJ03-5 MIDIOUT, SamacSys_Parts:KDJ035, symbol SamacSys_Parts:KDJ03-5
- added DgR8, DgR9: 220, Resistor_SMD:R_0805_2012Metric_Pad1.20x1.40mm_HandSolder, symbol Device:R
- added IC3: 74AHC1G04W5-7, SOT95P285X140-5N, symbol SamacSys_Parts:74AHC1G04W5-7
- added Q4: 2SC3325-Y, 2SC3325YLF, symbol SamacSys_Parts:2SC3325-Y
- DgJ8: value KDJ03-5 -> KDJ03-5 MIDIIN
Connections:
- net D+5V: now also DgR8.1, IC3.5 (VCC)
- net GNDD: now also DgJ1.2, DgJ1.MH1, DgJ1.MH2, IC3.3 (GND), Q4.2 (E)
- new net: IC3.4 (Y), Q4.1 (B)
- new net: DgR9.1, Q4.3 (C)
- new net: DgJ1.5, DgR9.2
- new net: DgJ1.4, DgR8.2
- new net D+5V_MIDITX: IC3.2 (A)
- no-connect marks 4 -> 6
Other:
- note added: "MIDI Interface Rx"
- note added: "MIDI Interface Tx"
- note removed: "MIDI Interface(RX only)"
