File: TBSEQ_Board_V3/mainBorad/mainBorad.kicad_pcb (KiCad board)
At the start: 2 copper layers, 258 parts, among them IC1 NJM2125F-TE1_DIP8, IC12 4066, IC2 NJM2125F-TE1_DIP8, IC4 NJM2125F-TE1, IC5 NJM2125F-TE1_DIP8, J1 Conn_01x08, J10 Conn_01x05, J11 Conn_01x05, J12 Conn_01x02, J13 Conn_01x01_Pin, J14 Conn_01x05, J2 Conn_01x05_Pin, J3 Conn_01x02_Pin, J4 Conn_01x03, J5 Conn_01x03, J6 MJ-462, J7 Conn_01x03_Pin, J8 Conn_01x02_Pin, J9 Conn_01x01_Pin, Q1 NPN, Q10 PNP, Q11 NPN, Q12 HN1C01FU-GR,LF, Q13 NPN, Q14 NPN, Q15 NPN, Q16 NPN, Q17 NPN, Q18 NPN, Q19 NPN, Q2 PNP, Q20 NPN, Q21 HN1C01FU-GR,LF, Q22 HN1C01FU-GR,LF, Q23 NPN, Q24 NPN, Q25 NPN, Q26 HN1C01FU-GR,LF, Q27 PNP, Q28 NJFET, Q29 NPN, Q30 NPN, Q35 NPN, Q36 PNP, Q37 NPN, Q38 PNP, Q39 NJFET, Q40 NPN, Q41 NPN, Q8 PNP, Q9 PNP, SW1 2MS1T1B4VS2QES, U1 LM13700

Commit message: V3Board
アートワーク中
Parts:
- removed J2: Conn_01x05_Pin, Connector_PinHeader_2.54mm:PinHeader_1x05_P2.54mm_Vertical
- added DgJ1: KDJ03-5 MIDIOUT, SamacSys_Parts:KDJ035, F.Cu at (107.4, 34.0)
- added DgR8: 220, Resistor_SMD:R_0805_2012Metric_Pad1.20x1.40mm_HandSolder, B.Cu at (107.6, 40.0)
- added DgR9: 220, Resistor_SMD:R_0805_2012Metric_Pad1.20x1.40mm_HandSolder, B.Cu at (112.1, 40.0)
- added IC3: 74AHC1G04W5-7, SamacSys_Parts:SOT95P285X140-5N, B.Cu at (117.5, 41.0)
- added Q4: 2SC3325-Y, SamacSys_Parts:2SC3325YLF, B.Cu at (112.4, 44.2)
- added VR1: RK09D117000B, SamacSys_Parts:RK09D117000B, F.Cu at (153.7, 67.9)
- DgC5, DgIC1, DgR1, DgR2, DgU2: moved to B.Cu
- DgIC2: value TC74VHC541FK -> 74VHC541FT; footprint SamacSys_Parts:SOP50P400X100-20N -> SamacSys_Parts:SOP65P640X120-20N
- DgIC3: value 74LVC541APW -> 74VHC541FT; footprint SamacSys_Parts:SOP65P640X110-20N -> SamacSys_Parts:SOP65P640X120-20N
- DgJ11: value MJ-8435 -> MJ-8435 CV OUT
- DgJ12: value MJ-8435 -> MJ-8435 GATE OUT
- DgJ13: value MJ-8435 -> MJ-8435 SYNC OUT
- DgJ8: value KDJ03-5 -> KDJ03-5 MIDIIN
- DgJ9: value MJ-8435 -> MJ-8435 SYNC IN
- IC2: value NJM2125F-TE1_DIP8 -> NJM2125F-TE1; footprint SamacSys_Parts:NJM2125F-SOT95&DIP8 -> SamacSys_Parts:SOT95P280X130-5N
- J4, J5: value Conn_01x03 -> Conn_01x02; footprint Connector_PinHeader_2.54mm:PinHeader_1x03_P2.54mm_Vertical -> Connector_PinHeader_2.54mm:PinHeader_1x02_P2.54mm_Vertical
- Q29, Q30, Q35, Q36, Q37, Q38, Q39, Q40, Q41: footprint Package_TO_SOT_THT:TO-92_Inline -> Package_TO_SOT_THT:TO-92_HandSolder
- moved J6 197.2 mm to (210.2, 29.9), turned to 180 degrees
- moved U1 192.9 mm to (219.1, 120.0), turned to -90 degrees
- moved C5 179.7 mm to (214.6, 106.7)
- moved R16 174.3 mm to (221.0, 84.9), turned to 90 degrees
- moved IC1 174.2 mm to (214.1, 80.6)
- moved VR8 169.6 mm to (222.5, 99.4), turned to 90 degrees
- moved R24 167.6 mm to (221.0, 79.4), turned to 90 degrees
- moved R14 164.4 mm to (219.1, 116.2), turned to 90 degrees
- moved R10 160.5 mm to (215.9, 116.2), turned to 90 degrees
- moved R9 157.4 mm to (212.7, 116.2), turned to 90 degrees
- moved R15 156.4 mm to (209.1, 106.7)
- moved VR9 154.3 mm to (221.8, 69.2), turned to 90 degrees
- moved R11 154.2 mm to (209.6, 116.2), turned to 90 degrees
- moved TM1 151.0 mm to (189.9, 114.9)
- moved DgR7 149.0 mm to (132.1, 60.3), turned to 90 degrees
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Connections:
- DgIC2 pad 13: Net-(DgIC2-Y6) -> D+5V_MIDITX
- DgIC2 pad 7: Net-(DgIC2-A6) -> D+3.3V_MIDITX
- DgJ3 pad 1: Net-(DgJ3-Pin_1) -> D+3.3V_MIDITX
- DgU1 pad 1: Net-(DgJ3-Pin_1) -> D+3.3V_MIDITX
- IC2 pad 1: A+VCO_CV -> A+CV
- IC2 pad 2: Net-(IC2--INPUT) -> GNDA
- IC2 pad 3: A+CV -> Net-(IC2--INPUT)
- IC2 pad 4: GNDA -> A+VCO_CV
- IC2 pad 5: unconnected-(IC2-NC-Pad5) -> A+12V
- J14 pad 4: A+TEMPO -> unconnected-(J14-Pin_4-Pad4)
- J4 pad 1: Net-(DgIC2-A6) -> Net-(DgIC2-A7)
- J4 pad 2: Net-(DgIC2-A7) -> Net-(DgIC2-A8)
- J5 pad 1: Net-(DgIC2-Y6) -> Net-(DgIC2-Y7)
- J5 pad 2: Net-(DgIC2-Y7) -> Net-(DgIC2-Y8)
Other:
- board outline added: 201 x 150 mm

Commit message: V3Board
アートワーク仮配置
Parts:
- Q1, Q10, Q11, Q13, Q14, Q15, Q16, Q17, Q18, Q19, Q2, Q20, Q23, Q24, Q25, Q27, Q28, Q8, Q9: footprint Package_TO_SOT_THT:TO-92_Inline -> Package_TO_SOT_THT:TO-92_HandSolder
- moved J12 107.4 mm to (219.1, 52.7), turned to -90 degrees
- moved R61 65.5 mm to (155.0, 110.5), turned to 180 degrees
- moved D1 62.4 mm to (154.2, 120.0), turned to 180 degrees
- moved D2 60.6 mm to (161.6, 110.5), turned to 180 degrees
- moved R26 60.2 mm to (167.5, 110.5), turned to 180 degrees
- moved TM3 59.1 mm to (86.4, 109.7), turned to 90 degrees
- moved Q1 57.6 mm to (164.5, 120.7), turned to -90 degrees
- moved C20 54.8 mm to (174.5, 126.3), turned to -90 degrees
- moved Q2 51.5 mm to (175.8, 121.3), turned to 180 degrees
- moved C17 51.3 mm to (72.9, 114.9)
- moved R46 50.5 mm to (140.3, 116.8)
- moved D3 49.9 mm to (167.3, 128.3), turned to 180 degrees
- moved R29 47.8 mm to (156.5, 128.3), turned to 180 degrees
- moved R25 46.9 mm to (169.5, 120.7), turned to -90 degrees
- moved R30 46.3 mm to (159.7, 128.3)
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
Commit message: V3Board
GNDパターン塗り済
Parts:
- removed J9: Conn_01x01_Pin, Connector_PinHeader_2.54mm:PinHeader_1x01_P2.54mm_Vertical
- C11, C13, C14, C15, C17, C22, C23, C29: footprint Capacitor_THT:CP_Radial_D5.0mm_P2.00mm -> Capacitor_THT:CP_Radial_D4.0mm_P2.00mm
- J14: footprint Connector_JST:JST_XH_S5B-XH-A-1_1x05_P2.50mm_Horizontal -> Connector_JST:JST_XH_B5B-XH-A_1x05_P2.50mm_Vertical
- moved J3 37.0 mm to (175.5, 113.0), turned to -90 degrees
- moved J14 32.8 mm to (64.9, 80.6), turned to 0 degrees
- moved VCA_R1 14.6 mm to (186.3, 135.0), turned to 90 degrees
- moved D2 13.3 mm to (162.2, 123.8)
- moved J7 13.3 mm to (159.0, 113.0), turned to 90 degrees
- moved R61 12.4 mm to (162.2, 120.7)
- moved VR5 11.6 mm to (138.9, 99.5)
- moved VR4 11.6 mm to (114.9, 98.6)
- moved SW1 11.6 mm to (33.7, 93.9)
- moved VR2 11.6 mm to (67.3, 99.5)
- moved VR3 11.6 mm to (91.3, 99.5)
- moved VR6 11.6 mm to (162.9, 99.4)
- moved VR7 11.6 mm to (186.9, 99.4)
- moved C3 11.5 mm to (179.3, 120.7)
- moved R94 11.0 mm to (134.0, 142.9), turned to 0 degrees
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- renumbered J1 to DgJ2
Connections:
- DgJ11 pad 2: A+CV_MIX -> A+VCO_CV
- DgJ11 pad 3: A+CV_MIX -> A+VCO_CV
- DgJ16 pad 2: A+CV_MIX -> A+VCO_CV
Routing:
- added copper zone on B.Cu, net ADAPTER GND
- added copper zone on F.Cu, net ADAPTER GND
- added copper zone on B.Cu, net GNDA
- added copper zone on F.Cu, net GNDA
- added copper zone on B.Cu, net GNDD
- added copper zone on F.Cu, net GNDD
Other:
- board size 201 x 150 mm -> 200 x 130.3 mm
- board text added: "A+ 12V"
- board text added: "A+ 5.3V"
- board text added: "AC C"
- board text added: "AUDIO OUT"
- board text added: "CV"
- board text added: "CV MX"
- board text added: "D+ 3V3"
- board text added: "D+ 5V"
- board text added: "ENV.M"
- board text added: "GA TE"
- board text added: "GNDA"
- board text added: "GNDD"
- board text added: "SL ID"
- board text added: "VCA.Env"
- board text added: "VCA.R"
- board text added: "VCA.RA"
- board text added: "VCA.Res"
- board text added: "VCA.Sig"
- board text added: "VCA.Tri"
