File: TBSEQ_Board_V3/mainBorad/VCF.kicad_sch (KiCad schematic)
At the start: 67 parts, among them J3 Conn_01x02_Pin, Q10 PNP, Q11 NPN, Q12 HN1C01FU-GR,LF, Q13 NPN, Q14 NPN, Q15 NPN, Q16 NPN, Q17 NPN, Q18 NPN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

Commit message: V3Board
DualTr フットプリント変更
配線ミス修正
TEMPO削除⇒PanelBoardに移動
Parts:
- Q12, Q21, Q22: footprint SamacSys_Parts:HN1C01FUGRLF -> SamacSys_Parts:HN1C01FUGRLF_SOT23&DIP8
Changed lines of the file:
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@@
 			)
 		)
-		(property "Footprint" "SamacSys_Parts:HN1C01FUGRLF"
+		(property "Footprint" "SamacSys_Parts:HN1C01FUGRLF_SOT23&DIP8"
 			(at 99.06 124.13 0)
 			(effects
@@
 			)
 		)
-		(property "Footprint" "SamacSys_Parts:HN1C01FUGRLF"
+		(property "Footprint" "SamacSys_Parts:HN1C01FUGRLF_SOT23&DIP8"
 			(at 97.79 213.03 0)
 			(effects
@@
 			)
 		)
-		(property "Footprint" "SamacSys_Parts:HN1C01FUGRLF"
+		(property "Footprint" "SamacSys_Parts:HN1C01FUGRLF_SOT23&DIP8"
 			(at 170.18 127.94 0)
 			(effects

Commit message: V3Board
アートワーク仮配置
Parts:
- Q10, Q11, Q13, Q14, Q15, Q16, Q17, Q18, Q19, Q20, Q23, Q9: footprint Package_TO_SOT_THT:TO-92_Inline -> Package_TO_SOT_THT:TO-92_HandSolder
Changed lines of the file:
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@@
 			)
 		)
-		(property "Footprint" "Package_TO_SOT_THT:TO-92_Inline"
+		(property "Footprint" "Package_TO_SOT_THT:TO-92_HandSolder"
 			(at 107.95 96.52 0)
 			(effects
@@
 			)
 		)
-		(property "Footprint" "Package_TO_SOT_THT:TO-92_Inline"
+		(property "Footprint" "Package_TO_SOT_THT:TO-92_HandSolder"
 			(at 133.35 158.75 0)
 			(effects
@@
 			)
 		)
-		(property "Footprint" "Package_TO_SOT_THT:TO-92_Inline"
+		(property "Footprint" "Package_TO_SOT_THT:TO-92_HandSolder"
 			(at 184.15 99.06 0)
 			(effects
@@
 			)
 		)
-		(property "Footprint" "Package_TO_SOT_THT:TO-92_Inline"
+		(property "Footprint" "Package_TO_SOT_THT:TO-92_HandSolder"
 			(at 199.39 39.37 0)
 			(effects
@@
 			)
 		)
-		(property "Footprint" "Package_TO_SOT_THT:TO-92_Inline"
+		(property "Footprint" "Package_TO_SOT_THT:TO-92_HandSolder"
 			(at 113.03 165.1 0)
 			(effects
@@
 			)
 		)
-		(property "Footprint" "Package_TO_SOT_THT:TO-92_Inline"
+		(property "Footprint" "Package_TO_SOT_THT:TO-92_HandSolder"
 			(at 83.82 96.52 0)
 			(effects
@@
 			)
 		)
-		(property "Footprint" "Package_TO_SOT_THT:TO-92_Inline"
+		(property "Footprint" "Package_TO_SOT_THT:TO-92_HandSolder"
 			(at 83.82 78.74 0)
 			(effects
@@
 			)
 		)
-		(property "Footprint" "Package_TO_SOT_THT:TO-92_Inline"
+		(property "Footprint" "Package_TO_SOT_THT:TO-92_HandSolder"
 			(at 107.95 78.74 0)
 			(effects
@@
 			)
 		)
-		(property "Footprint" "Package_TO_SOT_THT:TO-92_Inline"
+		(property "Footprint" "Package_TO_SOT_THT:TO-92_HandSolder"
 			(at 83.82 60.96 0)
 			(effects
@@
 			)
 		)
-		(property "Footprint" "Package_TO_SOT_THT:TO-92_Inline"
+		(property "Footprint" "Package_TO_SOT_THT:TO-92_HandSolder"
 			(at 107.95 60.96 0)
 			(effects
@@
 			)
 		)
-		(property "Footprint" "Package_TO_SOT_THT:TO-92_Inline"
+		(property "Footprint" "Package_TO_SOT_THT:TO-92_HandSolder"
 			(at 119.38 147.32 0)
 			(effects
@@
 			)
 		)
-		(property "Footprint" "Package_TO_SOT_THT:TO-92_Inline"
+		(property "Footprint" "Package_TO_SOT_THT:TO-92_HandSolder"
 			(at 147.32 64.77 0)
 			(effects

Commit message: V3Board
GNDパターン塗り済
Parts:
- C13, C14, C15, C17, C22, C23, C29: footprint Capacitor_THT:CP_Radial_D5.0mm_P2.00mm -> Capacitor_THT:CP_Radial_D4.0mm_P2.00mm
Changed lines of the file:
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@@
 			)
 		)
-		(property "Footprint" "Capacitor_THT:CP_Radial_D5.0mm_P2.00mm"
+		(property "Footprint" "Capacitor_THT:CP_Radial_D4.0mm_P2.00mm"
 			(at 234.95 87.63 0)
 			(effects
@@
 			)
 		)
-		(property "Footprint" "Capacitor_THT:CP_Radial_D5.0mm_P2.00mm"
+		(property "Footprint" "Capacitor_THT:CP_Radial_D4.0mm_P2.00mm"
 			(at 210.82 90.17 0)
 			(effects
@@
 			)
 		)
-		(property "Footprint" "Capacitor_THT:CP_Radial_D5.0mm_P2.00mm"
+		(property "Footprint" "Capacitor_THT:CP_Radial_D4.0mm_P2.00mm"
 			(at 203.2 50.8 0)
 			(effects
@@
 			)
 		)
-		(property "Footprint" "Capacitor_THT:CP_Radial_D5.0mm_P2.00mm"
+		(property "Footprint" "Capacitor_THT:CP_Radial_D4.0mm_P2.00mm"
 			(at 132.08 128.27 0)
 			(effects
@@
 			)
 		)
-		(property "Footprint" "Capacitor_THT:CP_Radial_D5.0mm_P2.00mm"
+		(property "Footprint" "Capacitor_THT:CP_Radial_D4.0mm_P2.00mm"
 			(at 166.37 60.96 0)
 			(effects
@@
 			)
 		)
-		(property "Footprint" "Capacitor_THT:CP_Radial_D5.0mm_P2.00mm"
+		(property "Footprint" "Capacitor_THT:CP_Radial_D4.0mm_P2.00mm"
 			(at 48.26 118.11 0)
 			(effects
@@
 			)
 		)
-		(property "Footprint" "Capacitor_THT:CP_Radial_D5.0mm_P2.00mm"
+		(property "Footprint" "Capacitor_THT:CP_Radial_D4.0mm_P2.00mm"
 			(at 157.48 101.6 0)
 			(effects

Commit message: V3Board
スペーサー穴追加
オートルーター後
DualTr,OPアンプは表面実装に切り替え
Parts:
- Q12, Q21, Q22: footprint SamacSys_Parts:HN1C01FUGRLF_SOT23&DIP8 -> SamacSys_Parts:HN1C01FUGRLF
Changed lines of the file:
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@@
 			)
 		)
-		(property "Footprint" "SamacSys_Parts:HN1C01FUGRLF_SOT23&DIP8"
+		(property "Footprint" "SamacSys_Parts:HN1C01FUGRLF"
 			(at 99.06 124.13 0)
 			(effects
@@
 			)
 		)
-		(property "Footprint" "SamacSys_Parts:HN1C01FUGRLF_SOT23&DIP8"
+		(property "Footprint" "SamacSys_Parts:HN1C01FUGRLF"
 			(at 97.79 213.03 0)
 			(effects
@@
 			)
 		)
-		(property "Footprint" "SamacSys_Parts:HN1C01FUGRLF_SOT23&DIP8"
+		(property "Footprint" "SamacSys_Parts:HN1C01FUGRLF"
 			(at 170.18 127.94 0)
 			(effects

Commit message: V3Board
DualTr OPAmp やはりDIPに変更してオートルーター前に戻す
Parts:
- Q12, Q21, Q22: footprint SamacSys_Parts:HN1C01FUGRLF -> SamacSys_Parts:HN1C01FUGRLF_DIP8
Changed lines of the file:
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@@
 			)
 		)
-		(property "Footprint" "SamacSys_Parts:HN1C01FUGRLF"
+		(property "Footprint" "SamacSys_Parts:HN1C01FUGRLF_DIP8"
 			(at 99.06 124.13 0)
 			(effects
@@
 			)
 		)
-		(property "Footprint" "SamacSys_Parts:HN1C01FUGRLF"
+		(property "Footprint" "SamacSys_Parts:HN1C01FUGRLF_DIP8"
 			(at 97.79 213.03 0)
 			(effects
@@
 			)
 		)
-		(property "Footprint" "SamacSys_Parts:HN1C01FUGRLF"
+		(property "Footprint" "SamacSys_Parts:HN1C01FUGRLF_DIP8"
 			(at 170.18 127.94 0)
 			(effects
