File: TBSEQ_Board_V3/panelBoard/Jack.kicad_sch (KiCad schematic)
At the start: 1 part, among them J1 Conn_01x05

Commit message: V3Board
PanelBoard⇒debugPanelBoardにして部品を全部表に出してアートワーク修正中
Parts:
- J1: footprint Connector_JST:JST_XH_B5B-XH-A_1x05_P2.50mm_Vertical -> Connector_PinSocket_2.54mm:PinSocket_1x05_P2.54mm_Vertical
Changed lines of the file:
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@@
 			)
 		)
-		(property "Footprint" "Connector_JST:JST_XH_B5B-XH-A_1x05_P2.50mm_Vertical"
+		(property "Footprint" "Connector_PinSocket_2.54mm:PinSocket_1x05_P2.54mm_Vertical"
 			(at 83.82 49.53 0)
 			(effects
