File: TBSEQ_Board_V4/DigitalBorad/SwitchMatrix.kicad_sch (KiCad schematic)
At the start: 29 parts

Commit message: TBSEQ_BoardV4
Parts:
- removed S1: B3F-1000S, SamacSys_Parts:B3F1060, symbol SamacSys_Parts:B3F-1000S
- added S2: B3F-1000S, SamacSys_parts:B3F1060, symbol SamacSys_Parts:B3F-1000S
- S10: renamed from S9; footprint SamacSys_Parts:B3F1060 -> SamacSys_parts:B3F1060
- S11: renamed from S10; footprint SamacSys_Parts:B3F1060 -> SamacSys_parts:B3F1060
- S12: renamed from S11; footprint SamacSys_Parts:B3F1060 -> SamacSys_parts:B3F1060
- S13: renamed from S12; footprint SamacSys_Parts:B3F1060 -> SamacSys_parts:B3F1060
- S14: renamed from S13; footprint SamacSys_Parts:B3F1060 -> SamacSys_parts:B3F1060
- S15: renamed from S14; footprint SamacSys_Parts:B3F1060 -> SamacSys_parts:B3F1060
- S16: renamed from S15; footprint SamacSys_Parts:B3F1060 -> SamacSys_parts:B3F1060
- S17: renamed from S16; footprint SamacSys_Parts:B3F1060 -> SamacSys_parts:B3F1060
- S18: renamed from S17; footprint SamacSys_Parts:B3F1060 -> SamacSys_parts:B3F1060
- S19: renamed from S18; footprint SamacSys_Parts:B3F1060 -> SamacSys_parts:B3F1060
- S20: renamed from S19; footprint SamacSys_Parts:B3F1060 -> SamacSys_parts:B3F1060
- S21: renamed from S20; footprint SamacSys_Parts:B3F1060 -> SamacSys_parts:B3F1060
- S22: renamed from S21; footprint SamacSys_Parts:B3F1060 -> SamacSys_parts:B3F1060
- S23: renamed from S22; footprint SamacSys_Parts:B3F1060 -> SamacSys_parts:B3F1060
- S24, S25, S26, S27, S28, S29, S30: footprint SamacSys_Parts:B3F1060 -> SamacSys_parts:B3F1060
- S3: renamed from S2; footprint SamacSys_Parts:B3F1060 -> SamacSys_parts:B3F1060
- S4: renamed from S3; footprint SamacSys_Parts:B3F1060 -> SamacSys_parts:B3F1060
- S5: renamed from S4; footprint SamacSys_Parts:B3F1060 -> SamacSys_parts:B3F1060
- S6: renamed from S5; footprint SamacSys_Parts:B3F1060 -> SamacSys_parts:B3F1060
- S7: renamed from S6; footprint SamacSys_Parts:B3F1060 -> SamacSys_parts:B3F1060
- S8: renamed from S7; footprint SamacSys_Parts:B3F1060 -> SamacSys_parts:B3F1060
- S9: renamed from S8; footprint SamacSys_Parts:B3F1060 -> SamacSys_parts:B3F1060
Connections:
- net COM1/KS0: now also S2.1 (COM_1), S2.2 (COM_2)
- net RowK3: now also S2.3 (N.O._1), S2.4 (N.O._2)
Other:
- moved on the sheet: S10, S11, S12, S13, S14, S15, S16, S17, S18, S19, S20, S21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
