File: TBSEQ_Board_V4/rythemPanelBoard/HT16K33.kicad_sch (KiCad schematic)
At the start: 18 parts, among them U7 HT16K33_28SOP-A_

Commit message: TBSEQ_BoardV4
Parts:
- U7: footprint SOIC127P1031X264-28N -> SamacSys_parts:SOIC127P1031X264-28N
